File: hardware/kicad/carrier.kicad_pcb (KiCad board)
At the start: 2 copper layers, 105 x 95 mm, 116 parts, among them J1 MC-107DMS, J10 J_ADS_MAIN ADSBee J5, J11 J_ADS_GNSS ADSBee J4, J2 J_NTC 103AT-2, J3 J_BAT JST-PH 2mm, J4 J_THERM 60C NC, J5 J_GNSS GPS-18037 J5, J6 J_ESP_A support, J7 J_ESP_B power/UART, J8 J_ESP_C I2C, J9 J_ESP_D support, Q1 2N7002, Q2 2N7002, Q3 2N7002, Q4 2N7002, Q5 MMBT3904, SW1 POWER JS102011SAQN (2=common), SW2 MUTE JS102011SAQN (2=common), U1 TPS70933DBVR, U10 BMP581, U2 TUSB320LAIRWBR, U3 SN74LVC1G02DBVR, U4 BQ25606RGER, U5 TLV840CADL29DBVR 2.9V, U6 TPS61088RHLR, U7 TPS22975DSGR, U8 MAX17048G+T10, U9 SN74LVC1G17DBVR

Commit message: Cleanups.
Parts:
- moved C32 80.5 mm to (92.2, 57.1), turned to 180 degrees
- moved U1 79.9 mm to (91.6, 60.1), turned to 180 degrees
- moved C2 72.2 mm to (88.4, 64.5)
- moved U3 61.2 mm to (85.4, 61.3), turned to -90 degrees
- moved R2 60.9 mm to (87.9, 60.7), turned to -90 degrees
- moved C4 60.9 mm to (87.9, 55.9), turned to 0 degrees
- moved U2 58.2 mm to (85.0, 65.0), turned to 90 degrees
- moved TP3 57.8 mm to (102.1, 65.8)
- moved R3 54.1 mm to (84.1, 55.9), turned to 180 degrees
- moved C31 53.6 mm to (30.0, 68.1), turned to -90 degrees
- moved R10 53.1 mm to (26.9, 68.1), turned to -90 degrees
- moved C26 52.8 mm to (95.0, 49.5), turned to 90 degrees
- moved C3 51.2 mm to (81.5, 63.5)
- moved R19 46.4 mm to (65.5, 56.6), turned to -90 degrees
- moved U5 44.8 mm to (99.6, 61.7)
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Routing:
- net GND: track 95.8 -> 229.1 mm, vias 89 -> 53
- net VBUS_DET: track 75.6 -> 2.39 mm, vias 4 -> 0
- net USB_CC2: track 89.2 -> 26.9 mm
- net RAIL_5V: track 97.5 -> 150.7 mm
- net ILIM_SW: track 51.6 -> 4.57 mm, vias 2 -> 0
- net GNSS_PPS: track 81.2 -> 127.0 mm
- net PWR_EN: track 86.9 -> 45.5 mm, vias 5 -> 2
- net VBAT: track 99.4 -> 61.3 mm, vias 2 -> 0
- net ILIM_HI: track 8.99 -> 42.6 mm
- net ADS_COMMS_TX: track 68.6 -> 40.1 mm
- net I2C_SCL: track 64.9 -> 38.3 mm, vias 0 -> 2
- net GNSS_3V3: track 85.1 -> 111.1 mm
- net GNSS_TXO: track 84.7 -> 109.0 mm
- net GNSS_RXI: track 78.7 -> 102.1 mm
- net ADS_COMMS_RX: track 63.6 -> 40.3 mm
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- removed copper zone on F.Cu, net GND

Commit message: Next
Parts:
- J2, J3, J4: footprint Connector_JST:JST_PH_B2B-PH-K_1x02_P2.00mm_Vertical -> carrier:JST_PH_B2B-PH-K_1x02_P2.00mm_Vertical_R10
- MH1, MH2, MH3, MH4, MH5: footprint MountingHole:MountingHole_2.8mm -> carrier:MountingHole_2.8mm
- MH6, MH7, MH8: footprint MountingHole:MountingHole_6.5mm -> carrier:MountingHole_6.5mm_Pad11mm
- SW2: footprint carrier:SW-SMD_JS102011SAQN -> SW-SMD_JS102011SAQN
Routing:
- net USB_VBUS: track 144.2 -> 141.4 mm
- net GND: track 229.1 -> 227.6 mm
- net PWR_EN: track 45.5 -> 44.2 mm
- net GNSS_3V3: track 111.1 -> 110.2 mm
- net BUZZ_PWM: track 87.3 -> 88.1 mm
- net CHG_CE_N: track 32.2 -> 32.7 mm
- net GNSS_RXI: track 102.1 -> 101.6 mm
Other:
- rule solder_mask_min_width: 0.1 -> 0.1016

Commit message: Routing
Parts:
- SW2: footprint SW-SMD_JS102011SAQN -> carrier:SW-SMD_JS102011SAQN
- moved C25 44.4 mm to (50.3, 20.9), turned to -90 degrees
- moved TP7 34.2 mm to (42.7, 38.1)
- moved JP1 32.6 mm to (42.7, 35.1), turned to 180 degrees
- moved JP2 31.5 mm to (78.0, 57.9), turned to 180 degrees
- moved C27 21.7 mm to (53.5, 57.5)
- moved U8 21.7 mm to (56.0, 57.6)
- moved R29 15.2 mm to (46.7, 38.1)
- moved J2 14.1 mm to (43.9, 84.8)
- moved R30 12.4 mm to (50.2, 34.9)
- moved TP6 9.66 mm to (35.3, 76.5)
- moved R15 6.91 mm to (97.3, 81.5)
- moved R33 6.61 mm to (61.2, 83.7), turned to 180 degrees
- moved R20 5.98 mm to (59.7, 58.7)
- moved R35 5.24 mm to (51.3, 84.6), turned to 180 degrees
- moved R14 4.83 mm to (96.5, 79.2), turned to 0 degrees
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Connections:
- J1 pad A8: (no net) -> unconnected-(J1-SBU1-PadA8)
- J1 pad B8: (no net) -> unconnected-(J1-SBU2-PadB8)
- J10 pad 10: (no net) -> unconnected-(J10-Pin_10-Pad10)
- J10 pad 11: (no net) -> unconnected-(J10-Pin_11-Pad11)
- J10 pad 12: (no net) -> unconnected-(J10-Pin_12-Pad12)
- J10 pad 5: (no net) -> unconnected-(J10-Pin_5-Pad5)
- J10 pad 6: (no net) -> unconnected-(J10-Pin_6-Pad6)
- J10 pad 7: (no net) -> unconnected-(J10-Pin_7-Pad7)
- J10 pad 8: (no net) -> unconnected-(J10-Pin_8-Pad8)
- J10 pad 9: (no net) -> unconnected-(J10-Pin_9-Pad9)
- J5 pad 3: (no net) -> unconnected-(J5-Pin_3-Pad3)
- J5 pad 7: (no net) -> unconnected-(J5-Pin_7-Pad7)
- J5 pad 8: (no net) -> unconnected-(J5-Pin_8-Pad8)
- J6 pad 1: (no net) -> unconnected-(J6-Pin_1-Pad1)
- J6 pad 2: (no net) -> unconnected-(J6-Pin_2-Pad2)
- J6 pad 3: (no net) -> unconnected-(J6-Pin_3-Pad3)
- J6 pad 5: (no net) -> unconnected-(J6-Pin_5-Pad5)
- J6 pad 6: (no net) -> unconnected-(J6-Pin_6-Pad6)
- J6 pad 7: (no net) -> unconnected-(J6-Pin_7-Pad7)
- J6 pad 8: (no net) -> unconnected-(J6-Pin_8-Pad8)
- J9 pad 1: (no net) -> unconnected-(J9-Pin_1-Pad1)
- J9 pad 2: (no net) -> unconnected-(J9-Pin_2-Pad2)
- U1 pad 3: (no net) -> unconnected-(U1-EN-Pad3)
- U1 pad 4: (no net) -> unconnected-(U1-NC-Pad4)
- U2 pad 5: (no net) -> unconnected-(U2-ADDR-Pad5)
- U2 pad 6: (no net) -> unconnected-(U2-INT_N/OUT3-Pad6)
- U2 pad 9: (no net) -> unconnected-(U2-ID-Pad9)
- U4 pad 2: (no net) -> unconnected-(U4-NC-Pad2)
- U4 pad 7: (no net) -> unconnected-(U4-~{PG}-Pad7)
- U5 pad 4: (no net) -> unconnected-(U5-NC-Pad4)
- U5 pad 5: (no net) -> unconnected-(U5-CT-Pad5)
- U8 pad 5: (no net) -> unconnected-(U8-~{ALRT}-Pad5)
- U9 pad 1: (no net) -> unconnected-(U9-NC-Pad1)
Routing:
- net GND: track 227.6 -> 57.7 mm, vias 53 -> 90
- net ADS_5V: track 65.5 -> 22.6 mm
- net USB_CC1: track 64.9 -> 23.8 mm
- net VBAT: track 61.3 -> 93.3 mm
- net ESP_5V: track 49.8 -> 17.9 mm
- net GNSS_PPS: track 127.0 -> 98.9 mm
- net I2C_SDA: track 40.5 -> 14.3 mm
- net USB_VBUS: track 141.4 -> 115.3 mm
- net BUZZ_PWM: track 88.1 -> 62.4 mm
- net REGN: track 63.4 -> 43.5 mm, vias 3 -> 2
- net ADS_COMMS_TX: track 40.1 -> 56.6 mm
- net BOOST_FB: track 19.5 -> 3.20 mm
- net ESP_UART_RX: track 22.4 -> 6.26 mm
- net RAIL_5V: track 150.7 -> 135.8 mm
- net I2C_SCL: track 38.3 -> 23.5 mm, vias 2 -> 0
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- added copper zone on F.Cu, net GND

Commit message: Revise charger
Parts:
- removed C2: 4.7u 25V, Capacitor_SMD:C_0805_2012Metric
- removed C3, C4: 100n, Capacitor_SMD:C_0603_1608Metric
- removed C32: 1u 50V, Capacitor_SMD:C_0603_1608Metric
- removed Q1: 2N7002, Package_TO_SOT_SMD:SOT-23
- removed Q5: MMBT3904, Package_TO_SOT_SMD:SOT-23
- removed R1: 910k 1%, Resistor_SMD:R_0603_1608Metric
- removed R2, R3, R35: 10k, Resistor_SMD:R_0603_1608Metric
- removed R32: 1M, Resistor_SMD:R_0603_1608Metric
- removed R4: 560R 1% ILIM2 2.3A, Resistor_SMD:R_0603_1608Metric
- removed R5: 330R 1% ILIM 1.45A, Resistor_SMD:R_0603_1608Metric
- removed R7: 100k VSET 4.2V, Resistor_SMD:R_0603_1608Metric
- removed U1: TPS70933DBVR, Package_TO_SOT_SMD:SOT-23-5
- removed U2: TUSB320LAIRWBR, Package_DFN_QFN:Texas_X2QFN-12_1.6x1.6mm_P0.4mm
- removed U3: SN74LVC1G02DBVR, Package_TO_SOT_SMD:SOT-23-5
- added C33: 22u 25V, C_0805_2012Metric, F.Cu at (64.7, 72.1)
- added C34: 2.2u 25V, C_0603_1608Metric, F.Cu at (63.0, 80.5)
- added Q6: 2N7002, SOT-23, F.Cu at (50.3, 86.4)
- added R36: 100k, R_0603_1608Metric, F.Cu at (54.6, 85.2)
- C5: value 1u 50V -> 2.2u 25V
- C7: value 4.7u 25V -> 2.2u 25V; footprint Capacitor_SMD:C_0805_2012Metric -> C_0603_1608Metric
- C8: value 47n 25V -> 100n
- L1: value 2.2uH CKST0603 -> 1uH FXL0630-1R0-M
- Q2, Q3, Q4: value 2N7002 -> AO3401A
- R12: value 100k -> 1M
- R23, R31: value 1k -> 560R
- R6: value 330R 1% ICHG 2.05A -> 13k 1% IFAST 1.85A
- R8: value 10k 1% -> 15k 1% THM bias
- U4: value BQ25606RGER -> MAX77757JEFG420+T; footprint Package_DFN_QFN:Texas_RGE0024H_VQFN-24-1EP_4x4mm_P0.5mm_EP2.7x2.7mm -> FC2QFN-24_L3.0-W3.0-P0.40_MAX77757
- moved J4 19.0 mm to (42.7, 86.4)
- moved J3 17.8 mm to (42.7, 76.2), turned to 180 degrees
- moved TP4 17.4 mm to (33.3, 85.3), turned to 180 degrees
- moved R10 16.7 mm to (37.1, 84.6), turned to 90 degrees
- moved C11 15.9 mm to (55.4, 80.8), turned to 90 degrees
- moved F1 14.8 mm to (43.9, 79.8)
- moved C31 14.4 mm to (35.6, 84.6), turned to 90 degrees
- moved C7 13.7 mm to (56.3, 73.2), turned to 90 degrees
- moved TP1 13.0 mm to (48.3, 81.8)
- moved TP6 11.4 mm to (28.2, 85.3)
- moved J2 10.7 mm to (50.3, 76.2), turned to 180 degrees
- moved R6 10.4 mm to (55.9, 78.2), turned to 180 degrees
- moved C5 10.0 mm to (70.6, 76.5), turned to -90 degrees
- moved R8 7.19 mm to (63.0, 79.0), turned to 0 degrees
- moved C9 6.67 mm to (76.2, 76.7), turned to -90 degrees
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Connections:
- C6 pad 1: CHG_PMID -> CHG_BYP
- C7 pad 1: REGN -> CHG_VDD
- Q2 pad 2: GND -> VSYS
- Q2 pad 3: CHG_CE_N -> CHG_DIS
- Q3 pad 1: CHG_IND_G -> CHG_STAT_N
- Q3 pad 2: GND -> VSYS
- Q3 pad 3: LED_CHG_A -> LED_G_SW
- Q4 pad 1: CHG_CE_N -> CHG_INOK_N
- Q4 pad 2: GND -> VSYS
- Q4 pad 3: LED_FULL_A -> LED_R_SW
- R12 pad 1: REGN -> CHG_DIS
- R12 pad 2: CHG_CE_N -> GND
- R23 pad 1: REGN -> LED_R_SW
- R31 pad 1: REGN -> LED_G_SW
- R33 pad 1: REGN -> VSYS
- R6 pad 1: CHG_ICHG -> CHG_IFAST
- R8 pad 1: REGN -> CHG_PVL
- U4 pad 1: USB_VBUS -> CHG_BTST
- U4 pad 10: CHG_ICHG -> CHG_VDD
- U4 pad 12: CHG_VSET -> CHG_IFAST
- U4 pad 17: GND -> CHG_PVL
- U4 pad 19: CHG_SW -> GND
- U4 pad 2: unconnected-(U4-NC-Pad2) -> CHG_INOK_N
- U4 pad 21: CHG_BTST -> CHG_SW
- U4 pad 22: REGN -> CHG_BYP
- U4 pad 23: CHG_PMID -> USB_VBUS
- U4 pad 3: USB_DP -> CHG_STAT_N
- U4 pad 4: USB_DN -> USB_CC2
- U4 pad 5: CHG_STAT_N -> USB_CC1
- U4 pad 6: GND -> USB_DP
- U4 pad 7: unconnected-(U4-~{PG}-Pad7) -> USB_DN
- U4 pad 8: CHG_ILIM -> GND
- U4 pad 9: CHG_CE_N -> GND
Routing:
- net USB_VBUS: track 115.3 -> 44.5 mm
- net VBAT: track 93.3 -> 49.0 mm, vias 0 -> 2
- net REGN: track 43.5 -> 0.00 mm, vias 2 -> 0
- net ILIM_HI: track 38.2 -> 0.00 mm
- net THERM_OK: track 70.9 -> 37.1 mm
- net USB_CC1: track 23.8 -> 51.9 mm
- net LED_FULL_A: track 31.9 -> 3.85 mm, vias 1 -> 0
- net USB_3V3: track 28.0 -> 0.00 mm
- net CHG_INOK_N: track 0.00 -> 25.6 mm, vias 0 -> 2
- net CHG_CE_N: track 24.6 -> 0.00 mm, vias 3 -> 0
- net CHG_DIS: track 0.00 -> 23.7 mm, vias 0 -> 2
- net LED_CHG_A: track 22.3 -> 3.69 mm, vias 1 -> 0
- net USB_DP: track 58.1 -> 43.1 mm, vias 3 -> 2
- net LED_R_SW: track 0.00 -> 14.9 mm, vias 0 -> 2
- net GND: track 57.7 -> 42.8 mm, vias 90 -> 80
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
Commit message: Cleanups
Parts:
- removed MH5: MountingHole_2.8mm, carrier:MountingHole_2.8mm
- added C35: 10n, Capacitor_SMD:C_0603_1608Metric, F.Cu at (55.6, 73.5)
- added C36: 1n DNP snubber, Capacitor_SMD:C_0603_1608Metric, F.Cu at (80.8, 63.2)
- added C37: 100n, Capacitor_SMD:C_0603_1608Metric, F.Cu at (92.2, 72.4)
- added C38: 100n, Capacitor_SMD:C_0603_1608Metric, F.Cu at (41.6, 39.4)
- added C39: 100n, Capacitor_SMD:C_0603_1608Metric, F.Cu at (96.8, 59.9)
- added FID1: Fiducial, carrier:Fiducial_1mm_Mask2mm, F.Cu at (4.00, 25.4)
- added FID2: Fiducial, carrier:Fiducial_1mm_Mask2mm, F.Cu at (73.0, 4.00)
- added FID3: Fiducial, carrier:Fiducial_1mm_Mask2mm, F.Cu at (97.5, 85.5)
- added MH10: MountingHole_2.7mm_M2.5, MountingHole:MountingHole_2.7mm_M2.5, F.Cu at (6.60, 17.5)
- added MH11: MountingHole_2.7mm_M2.5, MountingHole:MountingHole_2.7mm_M2.5, F.Cu at (32.0, 17.5)
- added MH12: MountingHole_2.7mm_M2.5, MountingHole:MountingHole_2.7mm_M2.5, F.Cu at (98.3, 18.1)
- added MH13: MountingHole_2.7mm_M2.5, MountingHole:MountingHole_2.7mm_M2.5, F.Cu at (47.5, 64.2)
- added MH14: MountingHole_2.7mm_M2.5, MountingHole:MountingHole_2.7mm_M2.5, F.Cu at (75.3, 58.6)
- added Q7: AO3401A, Package_TO_SOT_SMD:SOT-23, F.Cu at (88.4, 76.5)
- added Q8: 2N7002, Package_TO_SOT_SMD:SOT-23, F.Cu at (88.9, 80.0)
- added Q9: 2N7002, Package_TO_SOT_SMD:SOT-23, F.Cu at (84.3, 76.5)
- added R37: 6.2k 1%, Resistor_SMD:R_0603_1608Metric, F.Cu at (54.2, 76.8)
- added R39: 2.2R DNP snubber, Resistor_SMD:R_0603_1608Metric, F.Cu at (83.8, 63.2)
- added R40: 10k, Resistor_SMD:R_0603_1608Metric, F.Cu at (93.0, 74.7)
- added R41: 100k, Resistor_SMD:R_0603_1608Metric, F.Cu at (85.1, 79.0)
- added R42: 1M, Resistor_SMD:R_0603_1608Metric, F.Cu at (81.5, 76.7)
- added R43: 1k, Resistor_SMD:R_0603_1608Metric, F.Cu at (47.1, 86.4)
- added R44: 1M, Resistor_SMD:R_0603_1608Metric, F.Cu at (37.1, 39.9)
- added R45: 1M, Resistor_SMD:R_0603_1608Metric, F.Cu at (39.4, 39.9)
- added R46: 1M, Resistor_SMD:R_0603_1608Metric, F.Cu at (90.7, 57.7)
- added R47: 1M, Resistor_SMD:R_0603_1608Metric, F.Cu at (89.2, 57.7)
- added U11: LM73100RPWR, carrier:VQFN-10_L2.0-W2.0-P0.45-HR_LM73100, F.Cu at (93.9, 57.1)
- added U12: LM73100RPWR, carrier:VQFN-10_L2.0-W2.0-P0.45-HR_LM73100, F.Cu at (39.4, 37.6)
- C1: value 1u 50V -> 1u 50V X7R
- C10, C13, C14, C18, C19, C20, C9: value 22u 25V -> 22u 10V X7R
- C11, C24, C25, C26, C6: value 10u 25V -> 10u 25V X7R
- C15, C5: value 2.2u 25V -> 2.2u 25V X7R
- C21, C23: value 10n prelim -> 10n
- C22: value 100p prelim -> 100p
- C33: value 22u 25V -> 10u 25V X7R; footprint C_0805_2012Metric -> Capacitor_SMD:C_0805_2012Metric
- C34, C7: value 2.2u 25V -> 2.2u 25V X7R; footprint C_0603_1608Metric -> Capacitor_SMD:C_0603_1608Metric
- D5: footprint LED_THT:LED_D3.0mm -> carrier:LED_D3.0mm
- F1: value 3A -> 5A 0466005.NRHF
- J2: value J_NTC 103AT-2 -> J_NTC 100k ENTC-EB-100K4262-02
- JP1: value JP_PWR_ESP REMOVE FOR USB -> JP_PWR_ESP
- JP2: value JP_PWR_ADS REMOVE FOR USB -> JP_PWR_ADS
- L1: footprint carrier:IND-SMD_L7.4-W6.6 -> carrier:IND-SMD_L7.0-W6.6_FXL0630
- MH1, MH2, MH3, MH4: value MountingHole_2.8mm -> MountingHole_2.7mm_M2.5; footprint carrier:MountingHole_2.8mm -> MountingHole:MountingHole_2.7mm_M2.5
- MH6, MH7, MH8: footprint carrier:MountingHole_6.5mm_Pad11mm -> MountingHole:MountingHole_6.5mm
- Q6: footprint SOT-23 -> Package_TO_SOT_SMD:SOT-23
- R12: value 1M -> 100k
- R16: value 150k prelim -> 220k
- R17: value 160k prelim -> 160k
- R18: value 10k prelim -> 6.8k
- R36: footprint R_0603_1608Metric -> Resistor_SMD:R_0603_1608Metric
- R6: value 13k 1% IFAST 1.85A -> 6.2k 1%
- R8: value 15k 1% THM bias -> 154k 1%
- SW1: value POWER JS102011SAQN (2=common) -> JS102011SAQN
- SW2: value MUTE JS102011SAQN (2=common) -> JS102011SAQN
- TP1, TP2, TP3, TP4, TP5, TP6, TP7: footprint TestPoint:TestPoint_Pad_D1.5mm -> carrier:TestPoint_Pad_D1.5mm
- U4: footprint FC2QFN-24_L3.0-W3.0-P0.40_MAX77757 -> carrier:FC2QFN-24_L3.0-W3.0-P0.40_MAX77757
- U7: footprint Package_SON:Texas_DSG0008A_WSON-8-1EP_2x2mm_P0.5mm_EP0.9x1.6mm -> carrier:Texas_DSG0008A_WSON-8-1EP_2x2mm_P0.5mm_EP0.9x1.6mm
- U8: footprint Package_DFN_QFN:TDFN-8-1EP_2x2mm_P0.5mm_EP0.8x1.2mm -> carrier:TDFN-8_L2.0-W2.0-P0.50-EP0.8x1.38_T822
- moved TP3 56.8 mm to (45.4, 68.7)
- moved U5 48.0 mm to (52.2, 67.8)
- moved R13 46.9 mm to (52.3, 70.7)
- moved C12 40.2 mm to (56.6, 64.5)
- moved C14 38.0 mm to (54.7, 64.3), turned to 90 degrees
- moved C23 23.6 mm to (100.3, 63.0), turned to 90 degrees
- moved R12 22.2 mm to (47.6, 89.7), turned to 180 degrees
- moved C24 21.9 mm to (97.4, 62.9), turned to 90 degrees
- moved U7 21.8 mm to (99.9, 66.1), turned to 90 degrees
- moved U10 21.6 mm to (40.4, 58.7)
- moved C30 21.5 mm to (41.3, 61.0), turned to 180 degrees
- moved C22 21.0 mm to (93.7, 62.6), turned to 90 degrees
- moved C10 19.9 mm to (62.0, 77.0), turned to 0 degrees
- moved JP2 19.3 mm to (97.3, 57.4), turned to 90 degrees
- moved C21 19.0 mm to (95.6, 62.6), turned to 90 degrees
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Connections:
- J4 pad 1: VSYS -> /Battery, thermal, power control/THERM_FEED
- JP1 pad 1: RAIL_5V -> ESP_5V_D
- JP2 pad 1: RAIL_5V -> ADS_5V_D
- R6 pad 2: GND -> CHG_IFAST_MID
Routing:
- net RAIL_5V: track 130.7 -> 207.3 mm, vias 4 -> 8
- net GND: track 42.8 -> 112.6 mm, vias 80 -> 66
- net USB_VBUS: track 44.5 -> 102.3 mm
- net SW_EN: track 32.1 -> 82.7 mm, vias 0 -> 3
- net PWR_EN: track 44.0 -> 84.5 mm, vias 2 -> 4
- net VSYS: track 105.4 -> 75.6 mm, vias 0 -> 28
- net I2C_SDA: track 14.3 -> 37.3 mm, vias 0 -> 2
- net GNSS_3V3: track 107.1 -> 84.4 mm
- net VBAT: track 49.0 -> 63.0 mm, vias 2 -> 5
- net USB_DN: track 60.2 -> 47.3 mm
- net USB_CC1: track 51.9 -> 40.2 mm
- net ADS_5V: track 22.5 -> 11.4 mm
- net BUZZ_PLUS: track 16.5 -> 6.11 mm
- net BUZZ_LIM: track 12.0 -> 2.33 mm
- net CHG_INOK_N: track 25.6 -> 34.9 mm
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- added copper zone on F.Cu, net BOOST_SW
- added copper zone on B.Cu, net CHG_SW
- added copper zone on F.Cu, net CHG_SW
- added copper zone on In2.Cu, net CHG_SW
- added copper zone on In1.Cu, net GND
- added copper zone on In2.Cu, net GND
- added copper zone on F.Cu, net USB_VBUS
- added copper zone on F.Cu, net VBAT
- added copper zone on F.Cu, net VSYS
- added copper zone on In2.Cu, net VSYS
Other:
- copper layers 2 -> 4
- rule pad_to_mask_clearance: 0 -> 0.0254
- board text added: "ADSBee 1090U"
- board text added: "BAT"
- board text added: "ESP32 1.47{dblquote} IPS"
- board text added: "GNSS MAX-M10S"
- board text added: "NTC"
- board text added: "Rev A 2026-09-30"
- board text added: "THERM"
- board text added: "airgrep"

Commit message: Switches
Parts:
- added C40: 100n, Capacitor_SMD:C_0603_1608Metric, F.Cu at (32.8, 65.3)
- added J12: CONTROLS, Connector_PinHeader_2.54mm:PinHeader_2x04_P2.54mm_Vertical, F.Cu at (27.4, 78.2)
- added R48: 100k, Resistor_SMD:R_0603_1608Metric, F.Cu at (21.6, 74.7)
- added R49: 100k, Resistor_SMD:R_0603_1608Metric, F.Cu at (21.6, 77.2)
- added R50: 100k, Resistor_SMD:R_0603_1608Metric, F.Cu at (21.6, 79.8)
- added R51: 100k, Resistor_SMD:R_0603_1608Metric, F.Cu at (21.6, 82.3)
- added R52: 100k, Resistor_SMD:R_0603_1608Metric, F.Cu at (34.8, 75.2)
- added R53: 100k, Resistor_SMD:R_0603_1608Metric, F.Cu at (34.8, 72.6)
- added R54: 100k, Resistor_SMD:R_0603_1608Metric, F.Cu at (34.8, 70.1)
- added R55: 100k, Resistor_SMD:R_0603_1608Metric, F.Cu at (34.8, 67.6)
- added SW3: K3-1280S-F1, carrier:SW-SMD_K3-1280S-F1, F.Cu at (4.83, 47.0)
- added U13: TCA9534PWR, Package_SO:TSSOP-16_4.4x5mm_P0.65mm, F.Cu at (27.4, 69.3)
- SW1, SW2: value JS102011SAQN -> K3-1280S-F1; footprint carrier:SW-SMD_JS102011SAQN -> carrier:SW-SMD_K3-1280S-F1
- moved SW2 0.33 mm to (4.83, 65.8)
- moved SW1 0.18 mm to (61.5, 90.6)
Connections:
- BZ1 pad 1: BUZZ_PLUS -> BUZZ_LIM
- SW2 pad 1: BUZZ_LIM -> unconnected-(SW2-Pad1)
- SW2 pad 2: BUZZ_PLUS -> BUZZ_ENABLE
Routing:
- net ESP_3V3: track 146.0 -> 213.0 mm, vias 3 -> 5
- net WIFI_ENABLE: track 0.00 -> 46.2 mm, vias 0 -> 3
- net CTRL_P3: track 0.00 -> 39.1 mm, vias 0 -> 2
- net CTRL_P6: track 0.00 -> 33.7 mm, vias 0 -> 2
- net BUZZ_ENABLE: track 0.00 -> 31.4 mm, vias 0 -> 3
- net CTRL_P2: track 0.00 -> 24.8 mm, vias 0 -> 2
- net CTRL_P7: track 0.00 -> 22.6 mm, vias 0 -> 2
- net I2C_SCL: track 32.3 -> 53.0 mm, vias 2 -> 3
- net I2C_SDA: track 37.3 -> 55.2 mm, vias 2 -> 3
- net CTRL_P5: track 0.00 -> 17.0 mm, vias 0 -> 2
- net CTRL_P4: track 0.00 -> 17.0 mm, vias 0 -> 2
- net GND: track 112.6 -> 123.5 mm, vias 66 -> 69
- net BUZZ_PLUS: track 6.11 -> 0.00 mm
- net BUZZ_LIM: track 2.33 -> 6.75 mm
Other:
- board text added: "C40"
- board text added: "J12 INPUTS"
- board text added: "Rev 1 controls: K3 switches, U13 I2C inputs, J12 expansion"
- board text added: "Rev A 2026-10-06"
- board text added: "SW1 POWER"
- board text added: "SW2 MUTE"
- board text added: "SW3 WIFI"
- board text added: "U13"
- board text removed: "Rev A 2026-09-30"
