File: hardware/kicad/carrier.kicad_pcb (KiCad board)
At the start: 4 copper layers, 105 x 95 mm, 142 parts, among them J1 MC-107DMS, J10 J_ADS_MAIN ADSBee J5, J11 J_ADS_GNSS ADSBee J4, J12 CONTROLS, J2 J_NTC 100k ENTC-EB-100K4262-02, J3 J_BAT JST-PH 2mm, J4 J_THERM 60C NC, J5 J_GNSS GPS-18037 J5, J6 J_ESP_A support, J7 J_ESP_B power/UART, J8 J_ESP_C I2C, J9 J_ESP_D support, Q2 AO3401A, Q3 AO3401A, Q4 AO3401A, Q6 2N7002, Q7 AO3401A, Q8 2N7002, Q9 2N7002, SW1 K3-1280S-F1, SW2 K3-1280S-F1, SW3 K3-1280S-F1, U10 BMP581, U11 LM73100RPWR, U12 LM73100RPWR, U13 TCA9534PWR, U4 MAX77757JEFG420+T, U5 TLV840CADL29DBVR 2.9V, U6 TPS61088RHLR, U7 TPS22975DSGR, U8 MAX17048G+T10, U9 SN74LVC1G17DBVR

Commit message: Next
Parts:
- added FB1: BLM31KN471SZ1L, Inductor_SMD:L_1206_3216Metric, F.Cu at (132.4, 120.8)
- C1: value 1u 50V X7R -> 4.7u 50V X7R; footprint Capacitor_SMD:C_0603_1608Metric -> Capacitor_SMD:C_0805_2012Metric
- C33: value 10u 25V X7R -> 22u 16V X7R; footprint Capacitor_SMD:C_0805_2012Metric -> Capacitor_SMD:C_1206_3216Metric
- moved C14 78.7 mm to (109.5, 120.7), turned to 180 degrees
- moved D3 76.4 mm to (144.3, 122.4), turned to 90 degrees
- moved R29 68.5 mm to (103.7, 76.1)
- moved R55 68.3 mm to (85.3, 113.5)
- moved R54 67.7 mm to (85.3, 115.3)
- moved R53 67.2 mm to (85.3, 117.0)
- moved C12 67.0 mm to (108.5, 107.0)
- moved R52 66.7 mm to (85.3, 118.8)
- moved TP1 65.3 mm to (100.9, 121.1)
- moved R28 65.0 mm to (59.8, 102.9)
- moved C38 64.7 mm to (93.2, 78.4)
- moved C8 64.7 mm to (119.4, 111.1)
- moved R45 64.7 mm to (90.8, 79.1)
- moved R46 64.7 mm to (142.0, 97.0)
- moved R47 64.7 mm to (140.5, 97.0)
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Connections:
- C1 pad 1: USB_VBUS -> USB_VBUS_J1
- D3 pad 1: USB_VBUS -> USB_VBUS_J1
- J1 pad A4: USB_VBUS -> USB_VBUS_J1
- J1 pad A9: USB_VBUS -> USB_VBUS_J1
- J1 pad B4: USB_VBUS -> USB_VBUS_J1
- J1 pad B9: USB_VBUS -> USB_VBUS_J1
Routing:
- net USB_VBUS: track 102.3 -> 13.1 mm, vias 5 -> 6
- net ESP_3V3: track 213.0 -> 193.0 mm, vias 5 -> 12
- net CTRL_P3: track 39.1 -> 19.7 mm, vias 2 -> 0
- net USB_VBUS_J1: track 0.00 -> 18.8 mm, vias 0 -> 2
- net CTRL_P2: track 24.8 -> 13.6 mm, vias 2 -> 0
- net GND: track 123.5 -> 112.7 mm, vias 69 -> 64
- net CTRL_P6: track 33.7 -> 24.4 mm, vias 2 -> 0
- net RAIL_5V: track 207.3 -> 213.9 mm, vias 8 -> 7
- net ADS_COMMS_TX: track 56.6 -> 51.4 mm
- net ESP_UART_RX: track 6.26 -> 11.2 mm
- net BUZZ_ENABLE: track 31.4 -> 27.7 mm, vias 3 -> 2
- net BOOST_5V: track 22.2 -> 25.2 mm
- net VSYS: track 75.6 -> 73.1 mm, vias 28 -> 29
- net USB_CC1: track 40.2 -> 41.8 mm
- net USB_CC2: track 45.1 -> 46.7 mm
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- added copper zone on B.Cu, net USB_VBUS
- added copper zone on In2.Cu, net USB_VBUS
- removed copper zone on B.Cu, net CHG_SW
Other:
- board text added: "J12"
- board text added: "MUTE"
- board text added: "POWER"
- board text added: "Rev ${REVISION} ${ISSUE_DATE}"
- board text added: "USB"
- board text added: "WIFI"
- board text removed: "J12 INPUTS"
- board text removed: "Rev A 2026-10-06"
- board text removed: "SW1 POWER"
- board text removed: "SW2 MUTE"
- board text removed: "SW3 WIFI"
- board text removed: "U13"
