File: hardware/kicad/battery_control.kicad_sch (KiCad schematic)
At the start: 17 parts, among them J3 J_BAT JST-PH 2mm, J4 J_THERM 60C NC, Q2 2N7002, SW1 POWER JS102011SAQN (2=common), U5 TLV840CADL29DBVR 2.9V

Commit message: Next
Parts:
- J3, J4: footprint Connector_JST:JST_PH_B2B-PH-K_1x02_P2.00mm_Vertical -> carrier:JST_PH_B2B-PH-K_1x02_P2.00mm_Vertical_R10
Changed lines of the file:
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@@
 			)
 		)
-		(property "Footprint" "Connector_JST:JST_PH_B2B-PH-K_1x02_P2.00mm_Vertical"
+		(property "Footprint" "carrier:JST_PH_B2B-PH-K_1x02_P2.00mm_Vertical_R10"
 			(at 30.48 80.01 0)
 			(hide yes)
@@
 			)
 		)
-		(property "Footprint" "Connector_JST:JST_PH_B2B-PH-K_1x02_P2.00mm_Vertical"
+		(property "Footprint" "carrier:JST_PH_B2B-PH-K_1x02_P2.00mm_Vertical_R10"
 			(at 30.48 39.37 0)
 			(hide yes)

Commit message: Routing
Parts:
- C31: KiLib_Generator (none) -> SMD_2terminal_chip_molded
- TP1, TP2, TP3, TP4, TP5, TP6: now left out of the parts list

Commit message: Revise charger
Parts:
- added Q6: 2N7002, Package_TO_SOT_SMD:SOT-23, symbol Transistor_FET:2N7002
- Q2: value 2N7002 -> AO3401A; symbol Transistor_FET:2N7002 -> Transistor_FET:AO3401A; LCSC C8545 -> C15127
- R12: value 100k -> 1M; LCSC C25803 -> C22935
Connections:
- net REGN is gone; now on net CHG_DIS: R12.1
- net GND: now also R12.2, Q6.2 (S); no longer Q2.2 (S)
- net VSYS: now also Q2.2 (S)
- net CHG_CE_N renamed CHG_DIS
- net CHG_DIS: now also Q6.1 (G); no longer R12.2
- new net BAT_TS: Q6.3 (D)
Changed lines of the file:
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@@
 		)
 	)
-	(global_label "CHG_CE_N"
+	(global_label "GND"
 		(shape bidirectional)
 		(at 149.86 83.82 270)
@@
 		)
 	)
-	(global_label "CHG_CE_N"
+	(global_label "CHG_DIS"
 		(shape bidirectional)
 		(at 121.92 74.93 90)
@@
 		)
 	)
-	(global_label "REGN"
+	(global_label "CHG_DIS"
 		(shape bidirectional)
 		(at 149.86 76.2 90)
@@
 		)
 	)
-	(global_label "GND"
+	(global_label "VSYS"
 		(shape bidirectional)
 		(at 121.92 85.09 270)
@@
 			)
 		)
-		(property "Value" "100k"
+		(property "Value" "1M"
 			(at 152.4 80.01 0)
 			(show_name no)
@@
 			)
 		)
-		(property "LCSC" "C25803"
+		(property "LCSC" "C22935"
 			(at 147.32 80.01 0)
 			(hide yes)
@@
 	)
 	(symbol
-		(lib_id "Transistor_FET:2N7002")
+		(lib_id "Transistor_FET:AO3401A")
 		(at 119.38 80.01 0)
 		(unit 1)
@@
 			)
 		)
-		(property "Value" "2N7002"
+		(property "Value" "AO3401A"
 			(at 119.38 87.63 0)
 			(show_name no)
@@
 			)
 		)
-		(property "Datasheet" "https://www.onsemi.com/pub/Collateral/NDS7002A-D.PDF"
+		(property "Datasheet" "http://www.aosmd.com/pdfs/datasheet/AO3401A.pdf"
 			(at 124.46 76.2 0)
 			(hide yes)
@@
 			)
 		)
-		(property "LCSC" "C8545"
+		(property "LCSC" "C15127"
 			(at 119.38 72.39 0)
 			(hide yes)
@@
 		)
 	)
+	(symbol
+		(lib_id "Transistor_FET:2N7002")
+		(at 180.34 80.01 0)
+		(unit 1)
+		(body_style 1)
+		(exclude_from_sim no)
+		(in_bom yes)
+		(on_board yes)
+		(in_pos_files yes)
+		(dnp no)
+		(property "Reference" "Q6"
+			(at 180.34 72.39 0)
+			(show_name no)
+			(do_not_autoplace no)
+			(effects
+				(font
+					(size 1.27 1.27)
+				)
+				(justify left)
+			)
+		)
+		(property "Value" "2N7002"
+			(at 180.34 87.63 0)
+			(show_name no)
+			(do_not_autoplace no)
+			(effects
+				(font
+					(size 1.27 1.27)
+				)
+				(justify left)
+			)
+		)
+		(property "Footprint" "Package_TO_SOT_SMD:SOT-23"
+			(at 185.42 78.11 0)
+			(hide yes)
+			(show_name no)
+			(do_not_autoplace no)
+			(effects
+				(font
+					(size 1.27 1.27)
+					(italic yes)
+				)
+				(justify left)
+			)
+		)
+		(property "Datasheet" "https://www.onsemi.com/pub/Collateral/NDS7002A-D.PDF"
+			(at 185.42 76.2 0)
+			(hide yes)
+			(show_name no)
+			(do_not_autoplace no)
+			(effects
+				(font
+					(size 1.27 1.27)
+				)
+				(justify left)
+			)
+		)
+		(property "Description" "0.115A Id, 60V Vds, N-Channel MOSFET, SOT-23"
+			(at 180.34 80.01 0)
+			(hide yes)
+			(show_name no)
+			(do_not_autoplace no)
+			(effects
+				(font
+					(size 1.27 1.27)
+				)
+			)
+		)
+		(property "LCSC" "C8545"
+			(at 180.34 72.39 0)
+			(hide yes)
+			(show_name no)
+			(do_not_autoplace no)
+			(effects
+				(font
+					(size 1.27 1.27)
+				)
+			)
+		)
+		(pin "1"
+		)
+		(pin "2"
+		)
+		(pin "3"
+		)
+		(instances
+			(project "carrier"
+				(path "/1d76d2ec-7795-4c71-8167-b1182c3ebc1d/70bb31ad-859e-4aa6-9d27-4818f29c93a4"
+					(reference "Q6")
+					(unit 1)
+				)
+			)
+		)
+	)
+	(global_label "CHG_DIS"
+		(shape bidirectional)
+		(at 175.26 80.01 180)
+		(effects
+			(font
+				(size 1.27 1.27)
+			)
+			(justify right)
+		)
+		(property "Intersheetrefs" "${INTERSHEET_REFS}"
+			(at 175.26 80.01 0)
+			(hide yes)
+			(show_name no)
+			(do_not_autoplace no)
+			(effects
+				(font
+					(size 1.27 1.27)
+				)
+			)
+		)
+	)
+	(global_label "GND"
+		(shape bidirectional)
+		(at 182.88 85.09 270)
+		(effects
+			(font
+				(size 1.27 1.27)
+			)
+			(justify right)
+		)
+		(property "Intersheetrefs" "${INTERSHEET_REFS}"
+			(at 182.88 85.09 0)
+			(hide yes)
+			(show_name no)
+			(do_not_autoplace no)
+			(effects
+				(font
+					(size 1.27 1.27)
+				)
+			)
+		)
+	)
+	(global_label "BAT_TS"
+		(shape bidirectional)
+		(at 182.88 74.93 90)
+		(effects
+			(font
+				(size 1.27 1.27)
+			)
+			(justify left)
+		)
+		(property "Intersheetrefs" "${INTERSHEET_REFS}"
+			(at 182.88 74.93 0)
+			(hide yes)
+			(show_name no)
+			(do_not_autoplace no)
+			(effects
+				(font
+					(size 1.27 1.27)
+				)
+			)
+		)
+	)

Commit message: Cleanups
Parts:
- added C37: 100n, Capacitor_SMD:C_0603_1608Metric, symbol Device:C
- added Q7: AO3401A, Package_TO_SOT_SMD:SOT-23, symbol Transistor_FET:AO3401A
- added Q8, Q9: 2N7002, Package_TO_SOT_SMD:SOT-23, symbol Transistor_FET:2N7002
- added R40: 10k, Resistor_SMD:R_0603_1608Metric, symbol Device:R
- added R41: 100k, Resistor_SMD:R_0603_1608Metric, symbol Device:R
- added R42: 1M, Resistor_SMD:R_0603_1608Metric, symbol Device:R
- added R43: 1k, Resistor_SMD:R_0603_1608Metric, symbol Device:R
- F1: value 3A -> 5A 0466005.NRHF; LCSC C182445 -> C57525
- J3, J4: now not fitted; now left out of the parts list
- R12: value 1M -> 100k; LCSC C22935 -> C25803
- SW1: value POWER JS102011SAQN (2=common) -> JS102011SAQN
- TP1, TP2, TP3, TP4, TP5, TP6: footprint TestPoint:TestPoint_Pad_D1.5mm -> carrier:TestPoint_Pad_D1.5mm
Connections:
- net GND: now also C37.1, Q8.2 (S), Q9.2 (S), R41.2
- net PWR_EN: now also Q7.1 (G), Q8.3 (D)
- net SW_EN: now also R40.1
- net USB_VBUS: now also R42.1
- net VSYS: now also R43.1; no longer J4.1 (Pin_1)
- new net HOLD: C37.2, Q7.2 (S), R40.2
- new net LATCH: Q7.3 (D), Q8.1 (G), Q9.3 (D), R41.1
- new net THERM_FEED: J4.1 (Pin_1), R43.2
- new net USB_G: Q9.1 (G), R42.2
Other:
- note added: "Battery input"
- note added: "Battery input, thermal interlock, power switch and latch"
- note added: "Power switch, 2.9 V supervisor, under-voltage latch"
- note added: "Test points"
- note added: "Thermal interlock"
- title: (none) -> Battery, thermal, power control
- moved on the sheet: C12, C31, F1, Q2, Q6, R10, R12, R13, SW1, TP1, TP2, TP3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

Commit message: Switches
Parts:
- SW1: value JS102011SAQN -> K3-1280S-F1; footprint carrier:SW-SMD_JS102011SAQN -> carrier:SW-SMD_K3-1280S-F1; symbol carrier:JS102011SAQN -> carrier:K3-1280S-F1; LCSC C221660 -> C92658
Changed lines of the file:
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@@
 	)
 	(symbol
-		(lib_id "carrier:JS102011SAQN")
+		(lib_id "carrier:K3-1280S-F1")
 		(at 144.78 91.44 90)
 		(mirror x)
@@
 			)
 		)
-		(property "Value" "JS102011SAQN"
+		(property "Value" "K3-1280S-F1"
 			(at 139.7 91.44 90)
 			(show_name no)
@@
 			)
 		)
-		(property "Footprint" "carrier:SW-SMD_JS102011SAQN"
+		(property "Footprint" "carrier:SW-SMD_K3-1280S-F1"
 			(at 144.78 91.44 0)
 			(hide yes)
@@
 			)
 		)
-		(property "Datasheet" "https://lcsc.com/product-detail/Others_C-K-JS102011SAQN_C221660.html"
+		(property "Datasheet" "https://www.lcsc.com/datasheet/C92658.pdf"
 			(at 144.78 91.44 0)
 			(hide yes)
@@
 			)
 		)
-		(property "LCSC" "C221660"
+		(property "LCSC" "C92658"
 			(at 144.78 91.44 0)
 			(hide yes)
