File: hardware/kicad/boost_switch.kicad_sch (KiCad schematic)
At the start: 21 parts, among them U6 TPS61088RHLR, U7 TPS22975DSGR

Commit message: Routing
Parts:
- TP7: now left out of the parts list

Commit message: Cleanups
Parts:
- added C36: 1n DNP snubber, Capacitor_SMD:C_0603_1608Metric, symbol Device:C
- added R39: 2.2R DNP snubber, Resistor_SMD:R_0603_1608Metric, symbol Device:R
- C13, C14, C18, C19, C20: value 22u 25V -> 22u 10V X7R; LCSC C45783 -> C907991
- C15: value 2.2u 25V -> 2.2u 25V X7R; LCSC C57895 -> C415535
- C21, C23: value 10n prelim -> 10n
- C22: value 100p prelim -> 100p
- C24: value 10u 25V -> 10u 25V X7R; LCSC C15850 -> C3039694
- R16: value 150k prelim -> 220k; LCSC C22807 -> C22961
- R17: value 160k prelim -> 160k
- R18: value 10k prelim -> 6.8k; LCSC C25804 -> C23212
- TP7: footprint TestPoint:TestPoint_Pad_D1.5mm -> carrier:TestPoint_Pad_D1.5mm
- U7: footprint Package_SON:Texas_DSG0008A_WSON-8-1EP_2x2mm_P0.5mm_EP0.9x1.6mm -> carrier:Texas_DSG0008A_WSON-8-1EP_2x2mm_P0.5mm_EP0.9x1.6mm
Connections:
- net BOOST_SW: now also R39.1
- net GND: now also C36.2
- new net BOOST_SNUB: C36.1, R39.2
Other:
- note added: "5 V boost (TPS61088) and load switch (TPS22975)"
- title: (none) -> 5V boost and load switch
- moved on the sheet: C13, C14, C15, C16, C17, C18, C19, C20, C21, C22, C23, C24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
