File: hardware/kicad/buzzer_baro.kicad_sch (KiCad schematic)
At the start: 9 parts, among them SW2 MUTE JS102011SAQN (2=common), U10 BMP581, U9 SN74LVC1G17DBVR

Commit message: Cleanups
Parts:
- SW2: value MUTE JS102011SAQN (2=common) -> JS102011SAQN
Connections:
- no-connect marks 1 -> 0
Other:
- note added: "Barometer"
- note added: "Buzzer"
- note added: "Buzzer and barometer"
- title: (none) -> Buzzer and barometer
- moved on the sheet: BZ1, C28, C29, C30, R27, R28, SW2, U9

Commit message: Switches
Parts:
- added C40: 100n, Capacitor_SMD:C_0603_1608Metric, symbol Device:C
- added J12: CONTROLS, Connector_PinHeader_2.54mm:PinHeader_2x04_P2.54mm_Vertical, symbol Connector_Generic:Conn_02x04_Odd_Even
- added R48, R49, R50, R51, R52, R53, R54, R55: 100k, Resistor_SMD:R_0603_1608Metric, symbol Device:R
- added SW3: K3-1280S-F1, carrier:SW-SMD_K3-1280S-F1, symbol carrier:K3-1280S-F1
- added U13: TCA9534PWR, Package_SO:TSSOP-16_4.4x5mm_P0.65mm, symbol Interface_Expansion:TCA9534
- SW2: value JS102011SAQN -> K3-1280S-F1; footprint carrier:SW-SMD_JS102011SAQN -> carrier:SW-SMD_K3-1280S-F1; symbol carrier:JS102011SAQN -> carrier:K3-1280S-F1; LCSC C221660 -> C92658
Connections:
- net BUZZ_LIM: now also BZ1.1; no longer SW2.1
- net ESP_3V3: now also C40.1, R48.1, R49.1, R50.1, R51.1, R52.1, R53.1, R54.1, R55.1, U13.16 (VDD)
- net GND: now also C40.2, J12.7 (Pin_7), J12.8 (Pin_8), SW3.3, U13.1 (A0), U13.2 (A1), U13.3 (A2), U13.8 (GND)
- net I2C_SCL: now also U13.14 (SCL)
- net I2C_SDA: now also U13.15 (SDA)
- net BUZZ_PLUS renamed BUZZ_ENABLE
- net BUZZ_ENABLE: now also R48.2, U13.4 (P0); no longer BZ1.1
- new net CTRL_P2: J12.1 (Pin_1), R50.2, U13.6 (P2)
- new net CTRL_P3: J12.2 (Pin_2), R51.2, U13.7 (P3)
- new net CTRL_P4: J12.3 (Pin_3), R52.2, U13.9 (P4)
- new net CTRL_P5: J12.4 (Pin_4), R53.2, U13.10 (P5)
- new net CTRL_P6: J12.5 (Pin_5), R54.2, U13.11 (P6)
- new net CTRL_P7: J12.6 (Pin_6), R55.2, U13.12 (P7)
- new net WIFI_ENABLE: R49.2, SW3.2, U13.5 (P1)
- no-connect marks 0 -> 3
Other:
- note added: "Buzzer, barometer and physical controls"
- note added: "MUTE: P0=0 silent; P0=1 permits PWM. Wi-Fi: P1=0 off; P1=1 on. Read at startup; hold last valid state on read failure."
- note added: "Rev 1 controls: I2C 0x20, polled inputs; INT unused. R48-R55 bias all inputs high. J12: dry contacts to GND only."
- note removed: "Buzzer and barometer"
- moved on the sheet: SW2
