File: hardware/kicad/carrier.kicad_sch (KiCad schematic)
At the start: 0 parts

Commit message: Revise charger
Other:
- sheet Charger BQ25606 renamed Charger MAX77757
Changed lines of the file:
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@@
 			(color 0 0 0 0)
 		)
-		(property "Sheetname" "Charger BQ25606"
+		(property "Sheetname" "Charger MAX77757"
 			(at 102.54 18.73 0)
 			(show_name no)

Commit message: Cleanups
Other:
- note added: "Airfrep carrier"
- note added: "Battery in, 5 A fuse 60 C thermostat interlock ON switch, 2.9 V supervisor under-voltage latch, USB wake"
- note added: "ESP_3V3, I2C, BUZZ_PWM"
- note added: "I2C"
- note added: "Li-ion powered carrier for ESP32, ADSBee 1090 and GNSS modules"
- note added: "MAX17048 fuel gauge on I2C Charging and full LEDs 5 V rail LED (DNP)"
- note added: "MAX77757 1-cell Li-ion charger with USB-C CC detect SYS power path, NTC via BAT_TS"
- note added: "Piezo, Schmitt driver, mute switch BMP581 barometer on I2C"
- note added: "RAIL_5V 5 V"
- note added: "Sockets: ESP32, ADSBee 1090, GNSS LM66100 ideal diode and jumper per 5 V feed, UART cross-link"
- note added: "TPS61088 boost to 5 V TPS22975 load switch enabled by PWR_EN"
- note added: "USB-C receptacle 5 V in, CC and D+/D- to charger TVS on VBUS, ESD on CC and data"
- note added: "USB_VBUS 5 V"
- note added: "VBAT, VSYS"
- note added: "VBAT, charger status"
- note added: "VSYS, PWR_EN"
- title: (none) -> Airfrep carrier

Commit message: Next
Other:
- note added: "airgrep carrier"
- note removed: "Airfrep carrier"
- title: Airfrep carrier -> airgrep carrier
Changed lines of the file:
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@@
 	(paper "A4")
 	(title_block
-		(title "Airfrep carrier")
+		(title "airgrep carrier")
 		(rev "A")
+		(comment 1 "commit ${GIT_COMMIT}")
 	)
 	(text "I2C"
@@
 		)
 	)
-	(text "Airfrep carrier"
+	(text "airgrep carrier"
 		(exclude_from_sim no)
 		(at 20.32 33.02 0)
