File: hardware/kicad/charger.kicad_sch (KiCad schematic)
At the start: 14 parts, among them J2 J_NTC 103AT-2, U4 BQ25606RGER

Commit message: Next
Parts:
- J2: footprint Connector_JST:JST_PH_B2B-PH-K_1x02_P2.00mm_Vertical -> carrier:JST_PH_B2B-PH-K_1x02_P2.00mm_Vertical_R10
Changed lines of the file:
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@@
 			)
 		)
-		(property "Footprint" "Connector_JST:JST_PH_B2B-PH-K_1x02_P2.00mm_Vertical"
+		(property "Footprint" "carrier:JST_PH_B2B-PH-K_1x02_P2.00mm_Vertical_R10"
 			(at 139.7 119.38 0)
 			(hide yes)

Commit message: Revise charger
Parts:
- removed R5: 330R 1% ILIM 1.45A, Resistor_SMD:R_0603_1608Metric, symbol Device:R
- removed R7: 100k VSET 4.2V, Resistor_SMD:R_0603_1608Metric, symbol Device:R
- removed U4: BQ25606RGER, Package_DFN_QFN:Texas_RGE0024H_VQFN-24-1EP_4x4mm_P0.5mm_EP2.7x2.7mm, symbol carrier:BQ25606RGER
- added C33: 22u 25V, Capacitor_SMD:C_0805_2012Metric, symbol Device:C
- added C34: 2.2u 25V, Capacitor_SMD:C_0603_1608Metric, symbol Device:C
- added U4: MAX77757JEFG420+T, carrier:FC2QFN-24_L3.0-W3.0-P0.40_MAX77757, symbol carrier:MAX77757JEFG420
- C5: value 1u 50V -> 2.2u 25V; LCSC C15849 -> C57895
- C7: value 4.7u 25V -> 2.2u 25V; footprint Capacitor_SMD:C_0805_2012Metric -> Capacitor_SMD:C_0603_1608Metric; LCSC C1779 -> C57895
- C8: value 47n 25V -> 100n; LCSC C1622 -> C14663
- J2: value J_NTC 103AT-2 -> J_NTC 100k B57164K0104
- L1: value 2.2uH CKST0603 -> 1uH FXL0630-1R0-M; LCSC C3002634 -> C167216
- R6: value 330R 1% ICHG 2.05A -> 14k 1% IFAST 2.0A; LCSC C23138 -> C22803
- R8: value 10k 1% -> 130k 1% THM bias; LCSC C25804 -> C22795
Connections:
- net BAT_TS: now also U4.11 (THM)
- net CHG_BTST: now also U4.1 (BST)
- net CHG_STAT_N: now also U4.3 (STAT)
- net CHG_SW: now also U4.20 (LX), U4.21 (LX)
- net GND: now also C33.2, C34.2, U4.18 (PGND), U4.19 (PGND), U4.8 (ENBST), U4.9 (GND)
- net USB_DN: now also U4.7 (DN)
- net USB_DP: now also U4.6 (DP)
- net USB_VBUS: now also U4.23 (CHGIN), U4.24 (CHGIN)
- net VBAT: now also U4.13 (BATT), U4.14 (BATT)
- net VSYS: now also U4.15 (SYS), U4.16 (SYS)
- net CHG_ICHG renamed CHG_IFAST
- net CHG_IFAST: now also U4.12 (IFAST)
- net CHG_PMID renamed CHG_BYP
- net CHG_BYP: now also C33.1, U4.22 (BYP)
- net REGN renamed CHG_PVL
- net CHG_PVL: now also C34.1, U4.17 (PVL); no longer C7.1
- new net CHG_INOK_N: U4.2 (INOKB)
- new net CHG_VDD: C7.1, U4.10 (VDD)
- new net USB_CC1: U4.5 (CC1)
- new net USB_CC2: U4.4 (CC2)
- no-connect marks 2 -> 0

Commit message: Cleanups
Parts:
- added C35: 10n, Capacitor_SMD:C_0603_1608Metric, symbol Device:C
- added R37: 6.2k 1%, Resistor_SMD:R_0603_1608Metric, symbol Device:R
- C10, C9: value 22u 25V -> 22u 10V X7R; LCSC C45783 -> C907991
- C11, C6: value 10u 25V -> 10u 25V X7R; LCSC C15850 -> C3039694
- C33: value 22u 25V -> 10u 25V X7R; LCSC C45783 -> C3039694
- C34, C5, C7: value 2.2u 25V -> 2.2u 25V X7R; LCSC C57895 -> C415535
- J2: value J_NTC 100k B57164K0104 -> J_NTC 100k ENTC-EB-100K4262-02; now not fitted; now left out of the parts list
- L1: footprint carrier:IND-SMD_L7.4-W6.6 -> carrier:IND-SMD_L7.0-W6.6_FXL0630
- R6: value 14k 1% IFAST 2.0A -> 6.2k 1%; LCSC C22803 -> C4260
- R8: value 130k 1% THM bias -> 154k 1%; LCSC C22795 -> C22881
Connections:
- net BAT_TS: now also C35.1
- net GND: now also C35.2, R37.2; no longer R6.2
- new net CHG_IFAST_MID: R37.1, R6.2
Other:
- note added: "Battery charger (MAX77757)"
- title: (none) -> Charger MAX77757
- moved on the sheet: C10, C11, C33, C34, C5, C6, C7, C8, C9, L1, R6, R8

Commit message: Next
Parts:
- C33: value 10u 25V X7R -> 22u 16V X7R; footprint Capacitor_SMD:C_0805_2012Metric -> Capacitor_SMD:C_1206_3216Metric; LCSC C3039694 -> C385906
Changed lines of the file:
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@@
 		(title "Charger MAX77757")
 		(rev "A")
+		(comment 1 "commit ${GIT_COMMIT}")
 	)
 	(text "Battery charger (MAX77757)"
@@
 			)
 		)
-		(property "Value" "10u 25V X7R"
+		(property "Value" "22u 16V X7R"
 			(at 121.92 107.95 0)
 			(show_name no)
@@
 			)
 		)
-		(property "Footprint" "Capacitor_SMD:C_0805_2012Metric"
+		(property "Footprint" "Capacitor_SMD:C_1206_3216Metric"
 			(at 119.38 106.68 0)
 			(hide yes)
@@
 			)
 		)
-		(property "Datasheet" ""
+		(property "Datasheet" "https://ds.yuden.co.jp/TYCOMPAS/ut/detail?pn=EMK316BB7226ML-T"
 			(at 119.38 106.68 0)
 			(hide yes)
@@
 			)
 		)
-		(property "LCSC" "C3039694"
+		(property "LCSC" "C385906"
 			(at 119.38 106.68 0)
 			(hide yes)
