File: hardware/kicad/gauge_status.kicad_sch (KiCad schematic)
At the start: 15 parts, among them Q3 2N7002, Q4 2N7002, Q5 MMBT3904, U8 MAX17048G+T10

Commit message: Routing
Parts:
- Q5: KiLib_Generator (none) -> package/gullwing
- R19, R20: now left out of the parts list
- R35: KiLib_Generator (none) -> SMD_2terminal_chip_molded

Commit message: Revise charger
Parts:
- removed Q5: MMBT3904, Package_TO_SOT_SMD:SOT-23, symbol Transistor_BJT:MMBT3904
- removed R32: 1M, Resistor_SMD:R_0603_1608Metric, symbol Device:R
- removed R35: 10k, Resistor_SMD:R_0603_1608Metric, symbol Device:R
- added R36: 100k, Resistor_SMD:R_0603_1608Metric, symbol Device:R
- Q3, Q4: value 2N7002 -> AO3401A; symbol Transistor_FET:2N7002 -> Transistor_FET:AO3401A; LCSC C8545 -> C15127
- R23, R31: value 1k -> 560R; LCSC C21190 -> C23204
Connections:
- net CHG_IND_G is gone; now on net CHG_STAT_N: Q3.1 (G)
- net GND: no longer Q3.2 (S), Q4.2 (S)
- net LED_CHG_A: no longer Q3.3 (D)
- net LED_FULL_A: no longer Q4.3 (D)
- net CHG_CE_N renamed CHG_INOK_N
- net CHG_INOK_N: now also R36.2
- removed net REGN: R23.1, R31.1, R33.1
- new net LED_G_SW: Q3.3 (D), R31.1
- new net LED_R_SW: Q4.3 (D), R23.1
- new net VSYS: Q3.2 (S), Q4.2 (S), R33.1, R36.1

Commit message: Cleanups
Parts:
- D4: now not fitted; now left out of the parts list
- D5: footprint LED_THT:LED_D3.0mm -> carrier:LED_D3.0mm; now not fitted; now left out of the parts list
- U8: footprint Package_DFN_QFN:TDFN-8-1EP_2x2mm_P0.5mm_EP0.8x1.2mm -> carrier:TDFN-8_L2.0-W2.0-P0.50-EP0.8x1.38_T822
Other:
- note added: "Fuel gauge"
- note added: "Fuel gauge (MAX17048) and status LEDs"
- note added: "Status LEDs"
- title: (none) -> Gauge and status
- moved on the sheet: C27, Q3, Q4, R19, R20, R23, R26, R31, R33, R36
