File: hardware/kicad/modules.kicad_sch (KiCad schematic)
At the start: 13 parts, among them J10 J_ADS_MAIN ADSBee J5, J11 J_ADS_GNSS ADSBee J4, J5 J_GNSS GPS-18037 J5, J6 J_ESP_A support, J7 J_ESP_B power/UART, J8 J_ESP_C I2C, J9 J_ESP_D support

Commit message: Cleanups
Parts:
- added C38, C39: 100n, Capacitor_SMD:C_0603_1608Metric, symbol Device:C
- added R44, R45, R46, R47: 1M, Resistor_SMD:R_0603_1608Metric, symbol Device:R
- added U11, U12: LM73100RPWR, carrier:VQFN-10_L2.0-W2.0-P0.45-HR_LM73100, symbol carrier:LM73100RPW
- C25, C26: value 10u 25V -> 10u 25V X7R; LCSC C15850 -> C3039694
- J10, J11, J5, J6, J7, J8, J9: now not fitted; now left out of the parts list
- JP1: value JP_PWR_ESP REMOVE FOR USB -> JP_PWR_ESP; now not fitted; now left out of the parts list
- JP2: value JP_PWR_ADS REMOVE FOR USB -> JP_PWR_ADS; now not fitted; now left out of the parts list
Connections:
- net GND: now also C38.2, C39.2, R45.2, R47.2, U11.2 (OVLO), U11.4 (PGTH), U11.8 (GND), U11.9 (IMON), U12.2 (OVLO), U12.4 (PGTH), U12.8 (GND), U12.9 (IMON)
- net RAIL_5V: now also C38.1, C39.1, R44.1, R46.1, U11.5 (IN), U12.5 (IN); no longer JP1.1 (Pin_1), JP2.1 (Pin_1)
- new net ADS_5V_D: JP2.1 (Pin_1), U11.6 (OUT)
- new net ADS_ID_EN: R46.2, R47.1, U11.1 (EN/UVLO)
- new net ESP_5V_D: JP1.1 (Pin_1), U12.6 (OUT)
- new net ESP_ID_EN: R44.2, R45.1, U12.1 (EN/UVLO)
- no-connect marks 20 -> 24
Other:
- note added: "3.3 V rails sourced by the modules"
- note added: "5 V feeds (ideal diodes, jumper per module)"
- note added: "ADSBee"
- note added: "ESP32 module"
- note added: "GNSS module"
- note added: "Module sockets and 5 V feeds"
- note added: "UART link"
- title: (none) -> Modules and service shunts
- moved on the sheet: C25, C26, R29, R30
