File: hardware/kicad/usb_input.kicad_sch (KiCad schematic)
At the start: 19 parts, among them J1 MC-107DMS, Q1 2N7002, U1 TPS70933DBVR, U2 TUSB320LAIRWBR, U3 SN74LVC1G02DBVR

Commit message: Routing
Parts:
- C2, C32: KiLib_Generator (none) -> SMD_2terminal_chip_molded
- J1: MPN MC-107DMS -> (none); Manufacturer Hanbo Electronic -> (none)
- U1: KiLib_Generator (none) -> package/gullwing; MPN TPS70933DBVR -> (none); Manufacturer Texas Instruments -> (none)

Commit message: Revise charger
Parts:
- removed C2: 4.7u 25V, Capacitor_SMD:C_0805_2012Metric, symbol Device:C
- removed C3, C4: 100n, Capacitor_SMD:C_0603_1608Metric, symbol Device:C
- removed C32: 1u 50V, Capacitor_SMD:C_0603_1608Metric, symbol Device:C
- removed Q1: 2N7002, Package_TO_SOT_SMD:SOT-23, symbol Transistor_FET:2N7002
- removed R1: 910k 1%, Resistor_SMD:R_0603_1608Metric, symbol Device:R
- removed R2, R3: 10k, Resistor_SMD:R_0603_1608Metric, symbol Device:R
- removed R4: 560R 1% ILIM2 2.3A, Resistor_SMD:R_0603_1608Metric, symbol Device:R
- removed U1: TPS70933DBVR, Package_TO_SOT_SMD:SOT-23-5, symbol Regulator_Linear:AP2112K-3.3
- removed U2: TUSB320LAIRWBR, Package_DFN_QFN:Texas_X2QFN-12_1.6x1.6mm_P0.4mm, symbol carrier:TUSB320LAIRWBR
- removed U3: SN74LVC1G02DBVR, Package_TO_SOT_SMD:SOT-23-5, symbol 74xGxx:74LVC1G02
Connections:
- no-connect marks 7 -> 2

Commit message: Cleanups
Parts:
- C1: value 1u 50V -> 1u 50V X7R; LCSC C15849 -> C105174
- D6, D7, D8, D9: MPN (none) -> H5VLD3B; Manufacturer (none) -> Zhuhai Hongjiacheng (R+O)
Other:
- note added: "USB-C input"
- title: (none) -> USB input
- moved on the sheet: C1, D3, D6, D7, D8, D9, J1

Commit message: Next
Parts:
- added FB1: BLM31KN471SZ1L, Inductor_SMD:L_1206_3216Metric, symbol Device:FerriteBead
- C1: value 1u 50V X7R -> 4.7u 50V X7R; footprint Capacitor_SMD:C_0603_1608Metric -> Capacitor_SMD:C_0805_2012Metric; LCSC C105174 -> C437557
Connections:
- net USB_VBUS: now also FB1.2; no longer C1.1, D3.1 (K), J1.A4 (VBUS), J1.A9 (VBUS), J1.B4 (VBUS), J1.B9 (VBUS)
- new net USB_VBUS_J1: C1.1, D3.1 (K), FB1.1, J1.A4 (VBUS), J1.A9 (VBUS), J1.B4 (VBUS), J1.B9 (VBUS)
Changed lines of the file:
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@@
 		(title "USB input")
 		(rev "A")
+		(comment 1 "commit ${GIT_COMMIT}")
 	)
 	(text "USB-C input"
@@
 	)
 	(junction
+		(at 99.06 53.34)
+		(diameter 0)
+		(color 0 0 0 0)
+	)
+	(junction
 		(at 109.22 81.28)
 		(diameter 0)
 		(color 0 0 0 0)
 	)
-	(junction
-		(at 73.66 53.34)
-		(diameter 0)
-		(color 0 0 0 0)
-	)
 	(no_connect
 		(at 60.96 104.14)
@@
 	(wire
 		(pts
+			(xy 110.49 53.34) (xy 114.3 53.34)
+		)
+		(stroke
+			(width 0)
+			(type default)
+		)
+	)
+	(wire
+		(pts
 			(xy 109.22 107.95) (xy 109.22 111.76)
+		)
+		(stroke
+			(width 0)
+			(type default)
+		)
+	)
+	(wire
+		(pts
+			(xy 99.06 53.34) (xy 102.87 53.34)
 		)
 		(stroke
@@
 					(size 1.27 1.27)
 				)
+			)
+		)
+	)
+	(global_label "USB_VBUS_J1"
+		(shape input)
+		(at 76.2 53.34 180)
+		(fields_autoplaced yes)
+		(effects
+			(font
+				(size 1.27 1.27)
+			)
+			(justify right)
+		)
+		(property "Intersheetrefs" "${INTERSHEET_REFS}"
+			(at 60.3939 53.34 0)
+			(hide yes)
+			(show_name no)
+			(do_not_autoplace no)
+			(effects
+				(font
+					(size 1.27 1.27)
+				)
+				(justify right)
 			)
 		)
@@
 			)
 		)
-		(property "Value" "1u 50V X7R"
+		(property "Value" "4.7u 50V X7R"
 			(at 101.6 62.23 0)
 			(show_name no)
@@
 			)
 		)
-		(property "Footprint" "Capacitor_SMD:C_0603_1608Metric"
+		(property "Footprint" "Capacitor_SMD:C_0805_2012Metric"
 			(at 99.06 60.96 0)
 			(hide yes)
@@
 			)
 		)
-		(property "LCSC" "C105174"
+		(property "LCSC" "C437557"
 			(at 99.06 60.96 0)
 			(hide yes)
@@
 	)
 	(symbol
+		(lib_id "Device:FerriteBead")
+		(at 106.68 53.34 90)
+		(unit 1)
+		(body_style 1)
+		(exclude_from_sim no)
+		(in_bom yes)
+		(on_board yes)
+		(in_pos_files yes)
+		(dnp no)
+		(property "Reference" "FB1"
+			(at 106.68 48.26 0)
+			(show_name no)
+			(do_not_autoplace no)
+			(effects
+				(font
+					(size 1.27 1.27)
+				)
+			)
+		)
+		(property "Value" "BLM31KN471SZ1L"
+			(at 109.474 57.404 90)
+			(show_name no)
+			(do_not_autoplace no)
+			(effects
+				(font
+					(size 1.27 1.27)
+				)
+			)
+		)
+		(property "Footprint" "Inductor_SMD:L_1206_3216Metric"
+			(at 106.68 53.34 90)
+			(hide yes)
+			(show_name no)
+			(do_not_autoplace no)
+			(effects
+				(font
+					(size 1.27 1.27)
+				)
+			)
+		)
+		(property "Datasheet" "https://www.lcsc.com/datasheet/C710518.pdf"
+			(at 106.68 53.34 0)
+			(hide yes)
+			(show_name no)
+			(do_not_autoplace no)
+			(effects
+				(font
+					(size 1.27 1.27)
+				)
+			)
+		)
+		(property "Description" "Ferrite bead 470 Ω at 100 MHz, 4 A, 20 mΩ: filters the charger buck ripple from the USB cable"
+			(at 106.68 53.34 0)
+			(hide yes)
+			(show_name no)
+			(do_not_autoplace no)
+			(effects
+				(font
+					(size 1.27 1.27)
+				)
+			)
+		)
+		(property "LCSC" "C710518"
+			(at 106.68 53.34 0)
+			(hide yes)
+			(show_name no)
+			(do_not_autoplace no)
+			(effects
+				(font
+					(size 1.27 1.27)
+				)
+			)
+		)
+		(pin "1"
+		)
+		(pin "2"
+		)
+		(instances
+			(project "carrier"
+				(path "/1d76d2ec-7795-4c71-8167-b1182c3ebc1d/8d582056-b074-472b-a300-fd21b59a9139"
+					(reference "FB1")
+					(unit 1)
+				)
+			)
+		)
+	)
+	(symbol
 		(lib_id "carrier:USB_VBUS")
-		(at 73.66 53.34 0)
+		(at 114.3 53.34 0)
 		(unit 1)
 		(body_style 1)
@@
 		(dnp no)
 		(property "Reference" "#PWR001"
-			(at 73.66 57.15 0)
+			(at 114.3 57.15 0)
 			(hide yes)
 			(show_name no)
@@
 		)
 		(property "Value" "USB_VBUS"
-			(at 73.66 49.53 0)
+			(at 114.3 49.53 0)
 			(show_name no)
 			(do_not_autoplace no)
@@
 		)
 		(property "Footprint" ""
-			(at 73.66 53.34 0)
+			(at 114.3 53.34 0)
 			(hide yes)
 			(show_name no)
@@
 		)
 		(property "Datasheet" ""
-			(at 73.66 53.34 0)
+			(at 114.3 53.34 0)
 			(hide yes)
 			(show_name no)
@@
 		)
 		(property "Description" "Power symbol creates a global label with name \"USB_VBUS\""
-			(at 73.66 53.34 0)
-			(hide yes)
-			(show_name no)
+			(at 114.3 53.34 0)
+			(hide yes)
+			(show_name no)
