File: hardware/carrier-ti-charger/carrier.kicad_pcb (KiCad board)
At the start: 4 copper layers, 105 x 95 mm, 184 parts, among them J1 MC-107DMS, J10 J_ADS_MAIN ADSBee J5, J11 J_ADS_GNSS ADSBee J4, J12 CONTROLS, J2 J_NTC 100k ENTC-EB-100K4262-02, J3 J_BAT JST-PH 2mm, J4 J_THERM 60C NC, J5 J_GNSS GPS-18037 J5, J6 J_ESP_A support, J7 J_ESP_B power/UART, J8 J_ESP_C I2C, J9 J_ESP_D support, Q10 2N7002, Q11 2N7002, Q12 2N7002, Q13 CSD17575Q3, Q2 AO3401A, Q3 AO3401A, Q4 AO3401A, Q7 AO3401A, Q8 2N7002, Q9 2N7002, SW1 K3-1280S-F1, SW2 K3-1280S-F1, SW3 K3-1280S-F1, SW4 RESET 6x6, U10 BMP580, U11 TPS259474LRPWR, U12 TPS259474LRPWR, U13 TCA9534PWR, U14 TPS259474LRPWR, U4 BQ25798RQMR, U5 TLV840CADL29DBVR 2.9V, U6 TPS61088RHLR, U7 TPS22975DSGR, U8 MAX17048G+T10, U9 SN74LVC1G17DBVR

Commit message: Other MH's.
Parts:
- removed MH6, MH7, MH8: MountingHole_6.5mm, MountingHole:MountingHole_6.5mm
- added MH6ANTGNSS: MountingHole_6.5mm_Pad, MountingHole:MountingHole_6.5mm_Pad, F.Cu at (88.9, 47.6)
- added MH7ADS1090: MountingHole_6.5mm_Pad, MountingHole:MountingHole_6.5mm_Pad, F.Cu at (108.0, 47.6)
- added MH8ADS980: MountingHole_6.5mm_Pad, MountingHole:MountingHole_6.5mm_Pad, F.Cu at (127.0, 47.6)
- MH1, MH2, MH3, MH4: value MountingHole_2.7mm_M2.5 -> MountingHole_2.7mm_M2.5_Pad_Via; footprint MountingHole:MountingHole_2.7mm_M2.5 -> MountingHole:MountingHole_2.7mm_M2.5_Pad_Via
- TP1: value VBAT -> +VBAT
- TP2: value VSYS -> +VSYS
- TP5: value USB_VBUS -> +VUSB
- TP7: value RAIL_5V -> +5V
- moved FID2 28.2 mm to (151.8, 49.5)
- moved FID1 14.9 mm to (55.9, 49.5)
- moved MH2 0.78 mm to (152.3, 43.1)
- moved MH4 0.75 mm to (152.3, 130.0)
- moved MH1 0.63 mm to (55.3, 43.1)
- moved MH3 0.63 mm to (55.3, 130.0)
Connections:
- net ADS_5V renamed +ADS_5V
- net ADS_5V_D renamed +ADS_5V_D
- net BOOST_5V renamed +BOOST_5V
- net ESP_3V3 renamed +ESP_3V3
- net ESP_5V renamed +ESP_5V
- net ESP_5V_D renamed +ESP_5V_D
- net GNSS_3V3 renamed +GNSS_3V3
- net RAIL_5V renamed +5V
- net USB_DN renamed USB_D-
- net USB_DP renamed USB_D+
- net USB_VBUS renamed +VUSB
- net USB_VBUS_J1 renamed +VUSB_J1
- net VBAT renamed +VBAT
- net VSYS renamed +VSYS
Routing:
- net GNSS_TXO: track 93.1 -> 91.5 mm
- net +VUSB: track 27.9 -> 26.5 mm
- net GNSS_RXI: track 96.0 -> 94.8 mm
- net CHG_PMID: track 27.3 -> 26.6 mm
- net U14_ILM: track 6.73 -> 6.08 mm
- net CHG_BTST1: track 13.1 -> 13.8 mm
- net GND: vias 71 -> 69
Other:
- rule pad_to_mask_clearance: 0.0254 -> 0.1016
- board text removed: "Bottom plate sits on the solder mask through a thermal pad (no mask opening: vias of several nets lie under it). Outline on Dwgs.User."
- board text removed: "Rev 1 controls: K3 switches, U13 I2C inputs, J12 expansion"
