File: hardware/carrier-ti-charger/carrier.kicad_pcb (KiCad board)
At the start: 4 copper layers, 105 x 95 mm, 214 parts, among them J1 MC-107DMS, J10 J_ADS_MAIN ADSBee J5, J11 J_ADS_GNSS ADSBee J4, J12 CONTROLS, J13 GNSS_ANT, J2 NTC, J3 BAT, J4 THERM, J6 J_ESP_A support, J7 J_ESP_B power/UART, J8 J_ESP_C I2C, J9 J_ESP_D support, Q10 2N7002, Q11 2N7002, Q12 2N7002, Q13 CSD17575Q3, Q14 AO3401A, Q15 2N7002, Q16 2N7002, Q2 AO3401A, Q3 AO3401A, Q4 AO3401A, Q7 AO3401A, Q8 2N7002, Q9 2N7002, SW1 K3-1280S-F1, SW2 K3-1280S-F1, SW3 K3-1280S-F1, SW4 RESET 6x6, SW5 ACTIVE_ANT, U10 BMP580, U11 TPS259474LRPWR, U12 TPS259474LRPWR, U13 TCA9534PWR, U14 TPS259474LRPWR, U15 FUSB303BTMX, U16 MAX-M10S-00B, U17 TLV9001IDBVR, U18 TPS7A0233PDBVR, U4 BQ25798RQMR, U5 TLV840CADL29DBVR 2.9V, U6 TPS61088RHLR, U7 TPS22975DSGR, U8 MAX17048G+T10, U9 SN74LVC1G17DBVR

Commit message: Polishing.
Parts:
- added J2: XIAO Plus power/UART/PWM, Connector_PinHeader_2.54mm:PinHeader_1x07_P2.54mm_Vertical, F.Cu at (101.5, 59.0)
- added J3: XIAO Plus I2C/spares, Connector_PinHeader_2.54mm:PinHeader_1x07_P2.54mm_Vertical, F.Cu at (116.2, 59.0)
- added R90: 5.1k, Resistor_SMD:R_0805_2012Metric_Pad1.20x1.40mm_HandSolder, F.Cu at (114.8, 95.8)
- added R91: 5.1k, Resistor_SMD:R_0805_2012Metric_Pad1.20x1.40mm_HandSolder, F.Cu at (114.8, 99.6)
- R19, R20: value 1.8k -> 1.43k
- REF**: moved to B.Cu
- moved TP7 53.3 mm to (147.6, 100.2)
- moved REF** 26.9 mm to (139.7, 74.8), turned to 180 degrees
- moved C52 14.9 mm to (91.1, 59.9)
- moved C25 14.9 mm to (87.0, 59.9)
- moved C51 14.9 mm to (89.0, 59.9)
- moved R30 12.0 mm to (103.1, 86.2)
- moved R29 11.8 mm to (103.1, 87.9)
- moved C40 0.74 mm to (81.8, 104.6)
- moved C30 0.54 mm to (92.1, 99.9)
- moved R71 0.51 mm to (89.2, 72.6)
- moved R75 0.51 mm to (92.7, 78.5)
- moved U12 0.51 mm to (90.3, 76.7)
- moved C38 0.51 mm to (88.1, 75.9)
- moved C54 0.51 mm to (90.8, 72.6)
- moved R44 0.51 mm to (87.9, 78.5)
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- renumbered J7 to J1, J12 to J10, J3 to J11, J2 to J12, J4 to J13, J1 to J14, J6 to J4, J11 to J5, J10 to J6, J13 to J7, J9 to J8, J8 to J9, JP4 to JP2, JP2 to JP3
Connections:
- J1 pad 4: GND -> /Modules and service shunts/XIAO_D10
- J4 pad 1: unconnected-(J6-Pin_1-Pad1) -> /Modules and service shunts/XIAO_D0
- J4 pad 2: unconnected-(J6-Pin_2-Pad2) -> /Modules and service shunts/XIAO_D1
- J4 pad 3: unconnected-(J6-Pin_3-Pad3) -> /Modules and service shunts/XIAO_D2
- J4 pad 4: GND -> /Modules and service shunts/XIAO_D3
- J4 pad 7: unconnected-(J6-Pin_7-Pad7) (its old number) -> /Modules and service shunts/XIAO_D6
- U10 pad 7: GND -> unconnected-(U10-INT-Pad7)
Routing:
- net I2C_SCL: track 92.3 -> 125.7 mm, vias 4 -> 5
- net I2C_SDA: track 102.6 -> 133.7 mm
- net GND: track 101.5 -> 82.8 mm, vias 95 -> 91
- net ESP_UART_TX: track 4.82 -> 19.3 mm
- net ESP_UART_RX: track 11.2 -> 25.2 mm
- net +ESP_5V: track 21.9 -> 30.2 mm
- net +ESP_5V_D: track 64.0 -> 70.8 mm
- net +ESP_3V3: track 258.8 -> 253.0 mm
- net ADS_COMMS_TX: track 51.4 -> 46.9 mm
- net +5V: track 144.8 -> 148.8 mm, vias 8 -> 7
- net /Modules and service shunts/XIAO_D6: track 0.00 -> 3.65 mm
- net /Modules and service shunts/XIAO_D3: track 0.00 -> 3.65 mm
- net /Modules and service shunts/XIAO_D2: track 0.00 -> 3.65 mm
- net /Modules and service shunts/XIAO_D1: track 0.00 -> 3.65 mm
- net /Modules and service shunts/XIAO_D0: track 0.00 -> 3.65 mm
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Other:
- board text added: "ESP32 1.47"
- board text added: "ESP32-S3 Plus"
- board text removed: "ESP32 1.47{dblquote} IPS"
- board text removed: "GNSS MAX-M10S"

Commit message: Polishing.
Parts:
- R59: value 80.6k 1% -> 82k 1%
- R70, R71, R72: value 1.65k -> 1.8k
- moved C48 6.35 mm to (115.1, 103.0), turned to 0 degrees
- turned L2 to -90 degrees
Connections:
- L2 pad 1: +VSYS -> BOOST_SW
- L2 pad 2: BOOST_SW -> +VSYS
Routing:
- net CHG_REGN: track 19.8 -> 19.0 mm
- net GND: vias 91 -> 94

Commit message: Polishing
Routing:
- net U14_ILM: track 5.79 -> 5.78 mm, vias 2 -> 0
