File: hardware/carrier-ti-charger/buzzer_baro.kicad_sch (KiCad schematic)
At the start: 19 parts, among them J12 CONTROLS, SW2 K3-1280S-F1, SW3 K3-1280S-F1, U10 BMP580, U13 TCA9534PWR, U9 SN74LVC1G17DBVR

Commit message: Address review findings.
Parts:
- added C66: 1u, Capacitor_SMD:C_0603_1608Metric, symbol Device:C
- added D15, D16: 1N4148WS, Diode_SMD:D_SOD-323, symbol Device:D_Schottky
- added R87: 10k, carrier:R_0402_1005Metric_NoSilk, symbol Device:R
- added R88, R89: 100k 1%, Resistor_SMD:R_0603_1608Metric, symbol Device:R
- R28: value 150R -> 1k; LCSC C22808 -> C21190
Connections:
- net +ESP_3V3: now also R88.1, R89.1
- net BUZZ_LIM: now also C66.1; no longer BZ1.1
- net GND: now also R87.2
- net GNSS_RESET_N: now also D15.2 (A); no longer U13.6 (P2)
- net GNSS_SAFEBOOT_N: now also D16.2 (A); no longer U13.7 (P3)
- new net BUZZ_AC: BZ1.1, C66.2, R87.1
- new net GNSS_RESET_DRV: D15.1 (K), R88.2, U13.6 (P2)
- new net GNSS_SAFEBOOT_DRV: D16.1 (K), R89.2, U13.7 (P3)
Other:
- note added: "Rev 1 controls: I2C 0x20, polled; INT unused. R48, R49, R52-R55 bias the inputs high. P2 GNSS_RESET_N, P3 GNSS_SAFEBOOT_N: high-Z by default, firmware drives them low only; D15, D16 block a high level. J12 pins 1 and 2 unused. J12: dry contacts to GND only."
- note removed: "Rev 1 controls: I2C 0x20, polled; INT unused. R48, R49, R52-R55 bias the inputs high. P2 GNSS_RESET_N, P3 GNSS_SAFEBOOT_N: high-Z by default, firmware drives them low only. J12 pins 1 and 2 unused. J12: dry contacts to GND only."
