File: hardware/carrier-ti-charger/battery_control.kicad_sch (KiCad schematic)
At the start: 26 parts, among them J3 J_BAT JST-PH 2mm, J4 J_THERM 60C NC, Q2 AO3401A, Q6 2N7002, Q7 AO3401A, Q8 2N7002, Q9 2N7002, SW1 K3-1280S-F1, U5 TLV840CADL29DBVR 2.9V

Commit message: TI charger
Parts:
- removed Q6: 2N7002, Package_TO_SOT_SMD:SOT-23, symbol Transistor_FET:2N7002
- added Q11: 2N7002, Package_TO_SOT_SMD:SOT-23, symbol Transistor_FET:2N7002
- added R69: 100k 1%, Resistor_SMD:R_0603_1608Metric, symbol Device:R
- C12, C31, C37: value 100n -> 100n 50V
- R12, R13, R41: value 100k -> 100k 1%
Connections:
- net GND: now also Q11.2 (S)
- net SW_EN: now also R69.1
- new net SW_ON_N: Q11.3 (D)
- new net SW_SENSE_G: Q11.1 (G), R69.2
Other:
- note added: "(U13 P7): low = slider on."
- note added: "POWER slider to the expander"

Commit message: Other MH's.
Parts:
- TP1: value VBAT -> +VBAT
- TP2: value VSYS -> +VSYS
- TP5: value USB_VBUS -> +VUSB
Connections:
- net USB_VBUS renamed +VUSB
- net VBAT renamed +VBAT
- net VSYS renamed +VSYS
Changed lines of the file:
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@@
 	)
 	(symbol
-		(lib_id "carrier:VSYS")
+		(lib_id "carrier:+VSYS")
 		(at 198.12 54.61 0)
 		(unit 1)
@@
 			)
 		)
-		(property "Value" "VSYS"
+		(property "Value" "+VSYS"
 			(at 198.12 50.8 0)
 			(show_name no)
@@
 			)
 		)
-		(property "Description" "Power symbol creates a global label with name \"VSYS\""
+		(property "Description" "Power symbol creates a global label with name \"+VSYS\""
 			(at 198.12 54.61 0)
 			(hide yes)
@@
 	)
 	(symbol
-		(lib_id "carrier:VSYS")
+		(lib_id "carrier:+VSYS")
 		(at 30.48 129.54 0)
 		(unit 1)
@@
 			)
 		)
-		(property "Value" "VSYS"
+		(property "Value" "+VSYS"
 			(at 30.48 125.73 0)
 			(show_name no)
@@
 			)
 		)
-		(property "Description" "Power symbol creates a global label with name \"VSYS\""
+		(property "Description" "Power symbol creates a global label with name \"+VSYS\""
 			(at 30.48 129.54 0)
 			(hide yes)
@@
 	)
 	(symbol
-		(lib_id "carrier:USB_VBUS")
+		(lib_id "carrier:+VUSB")
 		(at 165.1 135.89 0)
 		(unit 1)
@@
 			)
 		)
-		(property "Value" "USB_VBUS"
+		(property "Value" "+VUSB"
 			(at 165.1 132.08 0)
 			(show_name no)
@@
 			)
 		)
-		(property "Description" "Power symbol creates a global label with name \"USB_VBUS\""
+		(property "Description" "Power symbol creates a global label with name \"+VUSB\""
 			(at 165.1 135.89 0)
 			(hide yes)
@@
 			)
 		)
-		(property "Value" "USB_VBUS"
+		(property "Value" "+VUSB"
 			(at 53.34 139.7 0)
 			(hide yes)
@@
 			)
 		)
-		(property "Value" "VBAT"
+		(property "Value" "+VBAT"
 			(at 86.36 53.34 0)
 			(hide yes)
@@
 			)
 		)
-		(property "Value" "VSYS"
+		(property "Value" "+VSYS"
 			(at 53.34 129.54 0)
 			(hide yes)
@@
 			)
 		)
-		(property "Description" "Q9 gate from USB_VBUS"
+		(property "Description" "Q9 gate from +VUSB"
 			(at 176.53 135.89 0)
 			(hide yes)
@@
 	)
 	(symbol
-		(lib_id "carrier:VSYS")
+		(lib_id "carrier:+VSYS")
 		(at 33.02 76.2 0)
 		(unit 1)
@@
 			)
 		)
-		(property "Value" "VSYS"
+		(property "Value" "+VSYS"
 			(at 33.02 72.39 0)
 			(show_name no)
@@
 			)
 		)
-		(property "Description" "Power symbol creates a global label with name \"VSYS\""
+		(property "Description" "Power symbol creates a global label with name \"+VSYS\""
 			(at 33.02 76.2 0)
 			(hide yes)
@@
 	)
 	(symbol
-		(lib_id "carrier:VSYS")
+		(lib_id "carrier:+VSYS")
 		(at 93.98 78.74 0)
 		(unit 1)
@@
 			)
 		)
-		(property "Value" "VSYS"
+		(property "Value" "+VSYS"
 			(at 93.98 74.93 0)
 			(show_name no)
@@
 			)
 		)
-		(property "Description" "Power symbol creates a global label with name \"VSYS\""
+		(property "Description" "Power symbol creates a global label with name \"+VSYS\""
 			(at 93.98 78.74 0)
 			(hide yes)
@@
 	)
 	(symbol
-		(lib_id "carrier:USB_VBUS")
+		(lib_id "carrier:+VUSB")
 		(at 30.48 139.7 0)
 		(unit 1)
@@
 			)
 		)
-		(property "Value" "USB_VBUS"
+		(property "Value" "+VUSB"
 			(at 30.48 135.89 0)
 			(show_name no)
@@
 			)
 		)
-		(property "Description" "Power symbol creates a global label with name \"USB_VBUS\""
+		(property "Description" "Power symbol creates a global label with name \"+VUSB\""
 			(at 30.48 139.7 0)
 			(hide yes)
@@
 			)
 		)
-		(property "Description" "Thermostat lead feed: limits a short of the user-made J4 lead to VSYS / 1 kOhm (4.2 mA); 10 kOhm would starve the undervoltage latch (Q8 gate)"
+		(property "Description" "Thermostat lead feed: limits a short of the user-made J4 lead to +VSYS / 1 kOhm (4.2 mA); 10 kOhm would starve the undervoltage latch (Q8 gate)"
 			(at 40.64 76.2 0)
 			(hide yes)
@@
 	)
 	(symbol
-		(lib_id "carrier:VBAT")
+		(lib_id "carrier:+VBAT")
 		(at 71.12 53.34 0)
 		(unit 1)
@@
 			)
 		)
-		(property "Value" "VBAT"
+		(property "Value" "+VBAT"
 			(at 71.12 49.53 0)
 			(show_name no)
@@
 			)
 		)
-		(property "Description" "Power symbol creates a global label with name \"VBAT\""
+		(property "Description" "Power symbol creates a global label with name \"+VBAT\""
 			(at 71.12 53.34 0)
 			(hide yes)

Commit message: Add USB current detection.
Parts:
- J3: value J_BAT JST-PH 2mm -> BAT
- J4: value J_THERM 60C NC -> THERM
Changed lines of the file:
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@@
 			)
 		)
-		(property "Value" "J_THERM 60C NC"
+		(property "Value" "THERM"
 			(at 53.34 82.55 0)
 			(show_name no)
@@
 			)
 		)
-		(property "Value" "J_BAT JST-PH 2mm"
+		(property "Value" "BAT"
 			(at 31.75 48.26 0)
 			(show_name no)

Commit message: Consolidate bom.
Parts:
- C12, C31, C37: value 100n 50V -> 100n 16V; footprint Capacitor_SMD:C_0603_1608Metric -> carrier:C_0402_1005Metric_NoSilk; LCSC C14663 -> C1525; MPN (none) -> CL05B104KO5NNNC
Changed lines of the file:
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@@
 			)
 		)
-		(property "Value" "100n 50V"
+		(property "Value" "100n 16V"
 			(at 68.58 93.98 0)
 			(show_name no)
@@
 			)
 		)
-		(property "Footprint" "Capacitor_SMD:C_0603_1608Metric"
+		(property "Footprint" "carrier:C_0402_1005Metric_NoSilk"
 			(at 66.04 92.71 0)
 			(hide yes)
@@
 			)
 		)
-		(property "LCSC" "C14663"
+		(property "LCSC" "C1525"
+			(at 66.04 92.71 0)
+			(hide yes)
+			(show_name no)
+			(do_not_autoplace no)
+			(effects
+				(font
+					(size 1.27 1.27)
+				)
+			)
+		)
+		(property "MPN" "CL05B104KO5NNNC"
 			(at 66.04 92.71 0)
 			(hide yes)
@@
 			)
 		)
-		(property "Value" "100n 50V"
+		(property "Value" "100n 16V"
 			(at 180.34 59.69 0)
 			(show_name no)
@@
 			)
 		)
-		(property "Footprint" "Capacitor_SMD:C_0603_1608Metric"
+		(property "Footprint" "carrier:C_0402_1005Metric_NoSilk"
 			(at 177.8 58.42 0)
 			(hide yes)
@@
 			)
 		)
-		(property "LCSC" "C14663"
+		(property "LCSC" "C1525"
+			(at 177.8 58.42 0)
+			(hide yes)
+			(show_name no)
+			(do_not_autoplace no)
+			(effects
+				(font
+					(size 1.27 1.27)
+				)
+			)
+		)
+		(property "MPN" "CL05B104KO5NNNC"
 			(at 177.8 58.42 0)
 			(hide yes)
@@
 			)
 		)
-		(property "Value" "100n 50V"
+		(property "Value" "100n 16V"
 			(at 179.07 123.19 0)
 			(show_name no)
@@
 			)
 		)
-		(property "Footprint" "Capacitor_SMD:C_0603_1608Metric"
+		(property "Footprint" "carrier:C_0402_1005Metric_NoSilk"
 			(at 176.53 121.92 0)
 			(hide yes)
@@
 			)
 		)
-		(property "LCSC" "C14663"
+		(property "LCSC" "C1525"
 			(at 176.53 121.92 0)
 			(hide yes)
+			(show_name no)
+			(do_not_autoplace no)
+			(effects
+				(font
+					(size 1.27 1.27)
+				)
+			)
+		)
+		(property "MPN" "CL05B104KO5NNNC"
+			(at 176.53 121.92 0)
+			(hide yes)

Commit message: Polishing.
Parts:
- renumbered J3 to J11, J4 to J13
Changed lines of the file:
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@@
 		(in_pos_files yes)
 		(dnp yes)
-		(property "Reference" "J4"
+		(property "Reference" "J13"
 			(at 53.34 72.39 0)
 			(show_name no)
@@
 			(project "carrier"
 				(path "/1d76d2ec-7795-4c71-8167-b1182c3ebc1d/70bb31ad-859e-4aa6-9d27-4818f29c93a4"
-					(reference "J4")
+					(reference "J13")
 					(unit 1)
 				)
@@
 		(in_pos_files yes)
 		(dnp yes)
-		(property "Reference" "J3"
+		(property "Reference" "J11"
 			(at 31.75 45.72 0)
 			(show_name no)
@@
 			(project "carrier"
 				(path "/1d76d2ec-7795-4c71-8167-b1182c3ebc1d/70bb31ad-859e-4aa6-9d27-4818f29c93a4"
-					(reference "J3")
-					(unit 1)
-				)
+					(reference "J11")
+					(unit 1)
+				)

Commit message: Consolidate BOM, add GNSS listen to ESP.
Parts:
- C12, C31, C37: footprint carrier:C_0402_1005Metric_NoSilk -> Mark:C_0402_1005Metric_NoSilk
- J11, J13: footprint carrier:JST_PH_B2B-PH-K_1x02_P2.00mm_Vertical_R10 -> Mark:JST_PH_B2B-PH-K_1x02_P2.00mm_Vertical_R10
- SW1: footprint carrier:SW-SMD_K3-1280S-F1 -> Mark:SW-SMD_K3-1280S-F1; symbol carrier:K3-1280S-F1 -> Mark:K3-1280S-F1
- TP1, TP2, TP3, TP4, TP5, TP6: footprint carrier:TestPoint_Pad_D1.5mm -> Mark:TestPoint_Pad_D1.5mm
- U5: footprint carrier:SOT-23-5_L2.9-W1.6-P0.95-LS2.8-BR -> Mark:SOT-23-5_L2.9-W1.6-P0.95-LS2.8-BR; symbol carrier:TLV840CADL29DBVR -> Mark:TLV840CADL29DBVR
Changed lines of the file:
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@@
 			)
 		)
-		(property "Footprint" "carrier:TestPoint_Pad_D1.5mm"
+		(property "Footprint" "Mark:TestPoint_Pad_D1.5mm"
 			(at 53.34 149.86 0)
 			(hide yes)
@@
 	)
 	(symbol
-		(lib_id "carrier:+VSYS")
+		(lib_id "Mark:+VSYS")
 		(at 198.12 54.61 0)
 		(unit 1)
@@
 	)
 	(symbol
-		(lib_id "carrier:+VSYS")
+		(lib_id "Mark:+VSYS")
 		(at 30.48 129.54 0)
 		(unit 1)
@@
 			)
 		)
-		(property "Footprint" "carrier:TestPoint_Pad_D1.5mm"
+		(property "Footprint" "Mark:TestPoint_Pad_D1.5mm"
 			(at 218.44 92.71 0)
 			(hide yes)
@@
 	)
 	(symbol
-		(lib_id "carrier:+VUSB")
+		(lib_id "Mark:+VUSB")
 		(at 165.1 135.89 0)
 		(unit 1)
@@
 			)
 		)
-		(property "Footprint" "carrier:TestPoint_Pad_D1.5mm"
+		(property "Footprint" "Mark:TestPoint_Pad_D1.5mm"
 			(at 53.34 139.7 0)
 			(hide yes)
@@
 			)
 		)
-		(property "Footprint" "carrier:TestPoint_Pad_D1.5mm"
+		(property "Footprint" "Mark:TestPoint_Pad_D1.5mm"
 			(at 86.36 53.34 0)
 			(hide yes)
@@
 			)
 		)
-		(property "Footprint" "carrier:TestPoint_Pad_D1.5mm"
+		(property "Footprint" "Mark:TestPoint_Pad_D1.5mm"
 			(at 76.2 86.36 0)
 			(hide yes)
@@
 			)
 		)
-		(property "Footprint" "carrier:C_0402_1005Metric_NoSilk"
+		(property "Footprint" "Mark:C_0402_1005Metric_NoSilk"
 			(at 66.04 92.71 0)
 			(hide yes)
@@
 			)
 		)
-		(property "Footprint" "carrier:JST_PH_B2B-PH-K_1x02_P2.00mm_Vertical_R10"
+		(property "Footprint" "Mark:JST_PH_B2B-PH-K_1x02_P2.00mm_Vertical_R10"
 			(at 54.61 76.2 0)
 			(hide yes)
@@
 			)
 		)
-		(property "Footprint" "carrier:C_0402_1005Metric_NoSilk"
+		(property "Footprint" "Mark:C_0402_1005Metric_NoSilk"
 			(at 177.8 58.42 0)
 			(hide yes)
@@
 			)
 		)
-		(property "Footprint" "carrier:TestPoint_Pad_D1.5mm"
+		(property "Footprint" "Mark:TestPoint_Pad_D1.5mm"
 			(at 53.34 129.54 0)
 			(hide yes)
@@
 	)
 	(symbol
-		(lib_id "carrier:K3-1280S-F1")
+		(lib_id "Mark:K3-1280S-F1")
 		(at 144.78 91.44 90)
 		(mirror x)
@@
 			)
 		)
-		(property "Footprint" "carrier:SW-SMD_K3-1280S-F1"
+		(property "Footprint" "Mark:SW-SMD_K3-1280S-F1"
 			(at 144.78 91.44 0)
 			(hide yes)
@@
 			)
 		)
-		(property "Footprint" "carrier:C_0402_1005Metric_NoSilk"
+		(property "Footprint" "Mark:C_0402_1005Metric_NoSilk"
 			(at 176.53 121.92 0)
 			(hide yes)
@@
 	)
 	(symbol
-		(lib_id "carrier:+VSYS")
+		(lib_id "Mark:+VSYS")
 		(at 33.02 76.2 0)
 		(unit 1)
@@
 	)
 	(symbol
-		(lib_id "carrier:+VSYS")
+		(lib_id "Mark:+VSYS")
 		(at 93.98 78.74 0)
 		(unit 1)
@@
 			)
 		)
-		(property "Footprint" "carrier:JST_PH_B2B-PH-K_1x02_P2.00mm_Vertical_R10"
+		(property "Footprint" "Mark:JST_PH_B2B-PH-K_1x02_P2.00mm_Vertical_R10"
 			(at 33.02 53.34 0)
 			(hide yes)
@@
 	)
 	(symbol
-		(lib_id "carrier:+VUSB")
+		(lib_id "Mark:+VUSB")
 		(at 30.48 139.7 0)
 		(unit 1)
@@
 	)
 	(symbol
-		(lib_id "carrier:+VBAT")
+		(lib_id "Mark:+VBAT")
 		(at 71.12 53.34 0)
 		(unit 1)
@@
 	)
 	(symbol
-		(lib_id "carrier:TLV840CADL29DBVR")
+		(lib_id "Mark:TLV840CADL29DBVR")
 		(at 198.12 68.58 0)
 		(unit 1)
@@
 			)
 		)
-		(property "Footprint" "carrier:SOT-23-5_L2.9-W1.6-P0.95-LS2.8-BR"
+		(property "Footprint" "Mark:SOT-23-5_L2.9-W1.6-P0.95-LS2.8-BR"
 			(at 198.12 68.58 0)
 			(hide yes)
