File: hardware/carrier-ti-charger/boost_switch.kicad_sch (KiCad schematic)
At the start: 23 parts, among them U6 TPS61088RHLR, U7 TPS22975DSGR

Commit message: TI charger
Parts:
- added C53: 100n 50V, Capacitor_SMD:C_0603_1608Metric, symbol Device:C
- C15: value 2.2u 25V X7R -> 4.7u 16V X5R; LCSC C415535 -> C19666
- C16: value 100n -> 100n 50V
- C17: value 47n -> 47n 50V
Connections:
- net BOOST_5V: now also C53.1
- net GND: now also C53.2
Other:
- moved on the sheet: C23, C24, TP7, U7

Commit message: Other MH's.
Parts:
- TP7: value RAIL_5V -> +5V
Connections:
- net BOOST_5V renamed +BOOST_5V
- net RAIL_5V renamed +5V
- net VSYS renamed +VSYS
Changed lines of the file:
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@@
 	)
 	(symbol
-		(lib_id "carrier:RAIL_5V")
+		(lib_id "carrier:+5V")
 		(at 250.19 82.55 0)
 		(unit 1)
@@
 			)
 		)
-		(property "Value" "RAIL_5V"
+		(property "Value" "+5V"
 			(at 250.19 78.74 0)
 			(show_name no)
@@
 			)
 		)
-		(property "Description" "Power symbol creates a global label with name \"RAIL_5V\""
+		(property "Description" "Power symbol creates a global label with name \"+5V\""
 			(at 250.19 82.55 0)
 			(hide yes)
@@
 			)
 		)
-		(property "Value" "RAIL_5V"
+		(property "Value" "+5V"
 			(at 275.59 82.55 0)
 			(hide yes)
@@
 	)
 	(symbol
-		(lib_id "carrier:BOOST_5V")
+		(lib_id "carrier:+BOOST_5V")
 		(at 121.92 72.39 0)
 		(unit 1)
@@
 			)
 		)
-		(property "Value" "BOOST_5V"
+		(property "Value" "+BOOST_5V"
 			(at 121.92 68.58 0)
 			(show_name no)
@@
 			)
 		)
-		(property "Description" "Power symbol creates a global label with name \"BOOST_5V\""
+		(property "Description" "Power symbol creates a global label with name \"+BOOST_5V\""
 			(at 121.92 72.39 0)
 			(hide yes)
@@
 	)
 	(symbol
-		(lib_id "carrier:VSYS")
+		(lib_id "carrier:+VSYS")
 		(at 20.32 72.39 0)
 		(unit 1)
@@
 			)
 		)
-		(property "Value" "VSYS"
+		(property "Value" "+VSYS"
 			(at 20.32 68.58 0)
 			(show_name no)
@@
 			)
 		)
-		(property "Description" "Power symbol creates a global label with name \"VSYS\""
+		(property "Description" "Power symbol creates a global label with name \"+VSYS\""
 			(at 20.32 72.39 0)
 			(hide yes)

Commit message: Refine resistors.
Parts:
- L2: value 2.2uH CKST0603 -> 2.2uH FC-ALX4030D-2R2MT; footprint carrier:IND-SMD_L7.4-W6.6 -> carrier:IND-SMD_L4.2-W4.2_FC-ALX4030D; LCSC C3002634 -> C5370906
Other:
- moved on the sheet: C36, R39
Changed lines of the file:
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@@
 	)
 	(junction
-		(at 73.66 93.98)
+		(at 69.85 93.98)
 		(diameter 0)
 		(color 0 0 0 0)
@@
 	(wire
 		(pts
-			(xy 73.66 93.98) (xy 73.66 96.52)
+			(xy 69.85 93.98) (xy 69.85 115.57)
 		)
 		(stroke
@@
 	(wire
 		(pts
-			(xy 73.66 114.3) (xy 73.66 116.84)
+			(xy 69.85 133.35) (xy 69.85 135.89)
 		)
 		(stroke
@@
 	(wire
 		(pts
-			(xy 73.66 104.14) (xy 73.66 106.68)
+			(xy 69.85 123.19) (xy 69.85 125.73)
 		)
 		(stroke
@@
 	)
 	(label "BOOST_SNUB"
-		(at 73.66 105.41 0)
+		(at 69.85 124.46 0)
 		(effects
 			(font
@@
 	)
 	(global_label "PWR_EN"
-		(shape bidirectional)
+		(shape input)
 		(at 212.09 102.87 180)
 		(effects
@@
 	(symbol
 		(lib_id "power:GND")
-		(at 73.66 116.84 0)
+		(at 69.85 135.89 0)
 		(unit 1)
 		(body_style 1)
@@
 		(dnp no)
 		(property "Reference" "#PWR048"
-			(at 73.66 123.19 0)
+			(at 69.85 142.24 0)
 			(hide yes)
 			(show_name no)
@@
 		)
 		(property "Value" "GND"
-			(at 73.66 120.65 0)
+			(at 69.85 139.7 0)
 			(show_name no)
 			(do_not_autoplace no)
@@
 		)
 		(property "Footprint" ""
-			(at 73.66 116.84 0)
+			(at 69.85 135.89 0)
 			(hide yes)
 			(show_name no)
@@
 		)
 		(property "Datasheet" ""
-			(at 73.66 116.84 0)
+			(at 69.85 135.89 0)
 			(hide yes)
 			(show_name no)
@@
 		)
 		(property "Description" "Power symbol creates a global label with name \"GND\" , ground"
-			(at 73.66 116.84 0)
+			(at 69.85 135.89 0)
 			(hide yes)
 			(show_name no)
@@
 	(symbol
 		(lib_id "Device:C")
-		(at 73.66 110.49 0)
+		(at 69.85 129.54 0)
 		(unit 1)
 		(body_style 1)
@@
 		(dnp yes)
 		(property "Reference" "C36"
-			(at 71.12 109.22 0)
+			(at 67.31 128.27 0)
 			(show_name no)
 			(do_not_autoplace no)
@@
 		)
 		(property "Value" "1n DNP snubber"
-			(at 71.12 111.76 0)
+			(at 67.31 130.81 0)
 			(show_name no)
 			(do_not_autoplace no)
@@
 		)
 		(property "Footprint" "Capacitor_SMD:C_0603_1608Metric"
-			(at 73.66 110.49 0)
+			(at 69.85 129.54 0)
 			(hide yes)
 			(show_name no)
@@
 		)
 		(property "Datasheet" ""
-			(at 73.66 110.49 0)
+			(at 69.85 129.54 0)
 			(hide yes)
 			(show_name no)
@@
 		)
 		(property "Description" "Unpolarized capacitor"
-			(at 73.66 110.49 0)
+			(at 69.85 129.54 0)
 			(hide yes)
 			(show_name no)
@@
 		)
 		(property "LCSC" ""
-			(at 73.66 110.49 0)
+			(at 69.85 129.54 0)
 			(hide yes)
 			(show_name no)
@@
 			)
 		)
-		(property "Value" "2.2uH CKST0603"
+		(property "Value" "2.2uH FC-ALX4030D-2R2MT"
 			(at 63.5 95.25 0)
 			(show_name no)
@@
 			)
 		)
-		(property "Footprint" "carrier:IND-SMD_L7.4-W6.6"
+		(property "Footprint" "carrier:IND-SMD_L4.2-W4.2_FC-ALX4030D"
 			(at 63.5 93.98 0)
 			(hide yes)
@@
 			)
 		)
-		(property "Datasheet" "https://www.lcsc.com/datasheet/C3002634.pdf"
+		(property "Datasheet" "https://datasheet.lcsc.com/datasheet/pdf/4f0a80287f31a1fb9e399a39619e691e.pdf?productCode=C5370906"
 			(at 63.5 93.98 0)
 			(hide yes)
@@
 			)
 		)
-		(property "LCSC" "C3002634"
+		(property "LCSC" "C5370906"
 			(at 63.5 93.98 0)
 			(hide yes)
@@
 	(symbol
 		(lib_id "Device:R")
-		(at 73.66 100.33 0)
+		(at 69.85 119.38 0)
 		(unit 1)
 		(body_style 1)
@@
 		(dnp yes)
 		(property "Reference" "R39"
-			(at 72.39 99.06 0)
+			(at 68.58 118.11 0)
 			(show_name no)
 			(do_not_autoplace no)
@@
 		)
 		(property "Value" "2.2R DNP snubber"
-			(at 72.39 101.6 0)
+			(at 68.58 120.65 0)
 			(show_name no)
 			(do_not_autoplace no)
@@
 		)
 		(property "Footprint" "Resistor_SMD:R_0603_1608Metric"
-			(at 73.66 100.33 0)
+			(at 69.85 119.38 0)
 			(hide yes)
 			(show_name no)
@@
 		)
 		(property "Datasheet" ""
-			(at 73.66 100.33 0)
+			(at 69.85 119.38 0)
 			(hide yes)
 			(show_name no)
@@
 		)
 		(property "Description" "Resistor"
-			(at 73.66 100.33 0)
+			(at 69.85 119.38 0)
 			(hide yes)
 			(show_name no)
@@
 		)
 		(property "LCSC" ""
-			(at 73.66 100.33 0)
+			(at 69.85 119.38 0)
 			(hide yes)
 			(show_name no)

Commit message: Consolidate bom.
Parts:
- C16, C53: value 100n 50V -> 100n 16V; footprint Capacitor_SMD:C_0603_1608Metric -> carrier:C_0402_1005Metric_NoSilk; LCSC C14663 -> C1525; MPN (none) -> CL05B104KO5NNNC
Changed lines of the file:
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@@
 			)
 		)
-		(property "Value" "100n 50V"
+		(property "Value" "100n 16V"
 			(at 127 81.28 0)
 			(show_name no)
@@
 			)
 		)
-		(property "Footprint" "Capacitor_SMD:C_0603_1608Metric"
+		(property "Footprint" "carrier:C_0402_1005Metric_NoSilk"
 			(at 129.54 80.01 0)
 			(hide yes)
@@
 			)
 		)
-		(property "LCSC" "C14663"
+		(property "LCSC" "C1525"
+			(at 129.54 80.01 0)
+			(hide yes)
+			(show_name no)
+			(do_not_autoplace no)
+			(effects
+				(font
+					(size 1.27 1.27)
+				)
+			)
+		)
+		(property "MPN" "CL05B104KO5NNNC"
 			(at 129.54 80.01 0)
 			(hide yes)
@@
 			)
 		)
-		(property "Value" "100n 50V"
+		(property "Value" "100n 16V"
 			(at 82.55 88.9 90)
 			(show_name no)
@@
 			)
 		)
-		(property "Footprint" "Capacitor_SMD:C_0603_1608Metric"
+		(property "Footprint" "carrier:C_0402_1005Metric_NoSilk"
 			(at 82.55 91.44 0)
 			(hide yes)
@@
 			)
 		)
-		(property "LCSC" "C14663"
-			(at 82.55 91.44 0)
-			(hide yes)
+		(property "LCSC" "C1525"
+			(at 82.55 91.44 0)
+			(hide yes)
+			(show_name no)
+			(do_not_autoplace no)
+			(effects
+				(font
+					(size 1.27 1.27)
+				)
+			)
+		)
+		(property "MPN" "CL05B104KO5NNNC"
+			(at 82.55 91.44 0)
+			(hide yes)

Commit message: Polishing.
Connections:
- net +VSYS: now also L2.2; no longer L2.1
- net BOOST_SW: now also L2.1; no longer L2.2
Other:
- moved on the sheet: L2
Changed lines of the file:
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@@
 	(symbol
 		(lib_id "carrier:CKST0603-2.2UH_M")
-		(at 63.5 93.98 0)
+		(at 63.5 93.98 180)
 		(unit 1)
 		(body_style 1)

Commit message: Consolidate BOM, add GNSS listen to ESP.
Parts:
- C16, C53: footprint carrier:C_0402_1005Metric_NoSilk -> Mark:C_0402_1005Metric_NoSilk
- L2: footprint carrier:IND-SMD_L4.2-W4.2_FC-ALX4030D -> Mark:IND-SMD_L4.2-W4.2_FC-ALX4030D; symbol carrier:CKST0603-2.2UH_M -> Mark:CKST0603-2.2UH_M
- TP7: footprint carrier:TestPoint_Pad_D1.5mm -> Mark:TestPoint_Pad_D1.5mm
- U6: footprint carrier:VQFN-20_L4.6-W3.6-P0.50-BL -> Mark:VQFN-20_L4.6-W3.6-P0.50-BL; symbol carrier:TPS61088RHLR -> Mark:TPS61088RHLR
- U7: footprint carrier:Texas_DSG0008A_WSON-8-1EP_2x2mm_P0.5mm_EP0.9x1.6mm -> Mark:Texas_DSG0008A_WSON-8-1EP_2x2mm_P0.5mm_EP0.9x1.6mm; symbol carrier:TPS22975DSGR -> Mark:TPS22975DSGR
Changed lines of the file:
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@@
 	)
 	(global_label "PWR_EN"
-		(shape bidirectional)
+		(shape input)
 		(at 87.63 130.81 180)
 		(effects
@@
 	)
 	(symbol
-		(lib_id "carrier:+5V")
+		(lib_id "Mark:+5V")
 		(at 250.19 82.55 0)
 		(unit 1)
@@
 			)
 		)
-		(property "Footprint" "carrier:TestPoint_Pad_D1.5mm"
+		(property "Footprint" "Mark:TestPoint_Pad_D1.5mm"
 			(at 275.59 82.55 0)
 			(hide yes)
@@
 			)
 		)
-		(property "Footprint" "carrier:C_0402_1005Metric_NoSilk"
+		(property "Footprint" "Mark:C_0402_1005Metric_NoSilk"
 			(at 129.54 80.01 0)
 			(hide yes)
@@
 			)
 		)
-		(property "Footprint" "carrier:C_0402_1005Metric_NoSilk"
+		(property "Footprint" "Mark:C_0402_1005Metric_NoSilk"
 			(at 82.55 91.44 0)
 			(hide yes)
@@
 	)
 	(symbol
-		(lib_id "carrier:TPS22975DSGR")
+		(lib_id "Mark:TPS22975DSGR")
 		(at 229.87 101.6 0)
 		(unit 1)
@@
 			)
 		)
-		(property "Footprint" "carrier:Texas_DSG0008A_WSON-8-1EP_2x2mm_P0.5mm_EP0.9x1.6mm"
+		(property "Footprint" "Mark:Texas_DSG0008A_WSON-8-1EP_2x2mm_P0.5mm_EP0.9x1.6mm"
 			(at 229.87 101.6 0)
 			(hide yes)
@@
 	)
 	(symbol
-		(lib_id "carrier:TPS61088RHLR")
+		(lib_id "Mark:TPS61088RHLR")
 		(at 101.6 101.6 0)
 		(unit 1)
@@
 			)
 		)
-		(property "Footprint" "carrier:VQFN-20_L4.6-W3.6-P0.50-BL"
+		(property "Footprint" "Mark:VQFN-20_L4.6-W3.6-P0.50-BL"
 			(at 101.6 101.6 0)
 			(hide yes)
@@
 	)
 	(symbol
-		(lib_id "carrier:+BOOST_5V")
+		(lib_id "Mark:+BOOST_5V")
 		(at 121.92 72.39 0)
 		(unit 1)
@@
 	)
 	(symbol
-		(lib_id "carrier:CKST0603-2.2UH_M")
+		(lib_id "Mark:CKST0603-2.2UH_M")
 		(at 63.5 93.98 180)
 		(unit 1)
@@
 			)
 		)
-		(property "Footprint" "carrier:IND-SMD_L4.2-W4.2_FC-ALX4030D"
+		(property "Footprint" "Mark:IND-SMD_L4.2-W4.2_FC-ALX4030D"
 			(at 63.5 93.98 0)
 			(hide yes)
@@
 	)
 	(symbol
-		(lib_id "carrier:+VSYS")
+		(lib_id "Mark:+VSYS")
 		(at 20.32 72.39 0)
 		(unit 1)
