File: hardware/carrier-ti-charger/gauge_status.kicad_sch (KiCad schematic)
At the start: 13 parts, among them Q3 AO3401A, Q4 AO3401A, U8 MAX17048G+T10

Commit message: TI charger
Parts:
- C27: value 100n -> 100n 50V
- R23, R31: value 560R -> 470R; LCSC C23204 -> C23179
- R33: value 47k -> 47k 1%
- R36: value 100k -> 100k 1%
Connections:
- net CHG_INOK_N renamed USB_OK_N
Changed lines of the file:
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@@
 		)
 	)
-	(global_label "CHG_INOK_N"
+	(global_label "USB_OK_N"
 		(shape bidirectional)
 		(at 68.58 99.06 180)
@@
 			)
 		)
-		(property "Value" "100k"
+		(property "Value" "100k 1%"
 			(at 74.93 92.71 0)
 			(show_name no)
@@
 			)
 		)
-		(property "Value" "100n"
+		(property "Value" "100n 50V"
 			(at 175.26 90.17 0)
 			(show_name no)
@@
 			)
 		)
-		(property "Value" "560R"
+		(property "Value" "470R"
 			(at 113.03 115.57 0)
 			(show_name no)
@@
 			)
 		)
-		(property "LCSC" "C23204"
+		(property "LCSC" "C23179"
 			(at 111.76 114.3 0)
 			(hide yes)
@@
 			)
 		)
-		(property "Value" "560R"
+		(property "Value" "470R"
 			(at 105.41 115.57 0)
 			(show_name no)
@@
 			)
 		)
-		(property "LCSC" "C23204"
+		(property "LCSC" "C23179"
 			(at 106.68 114.3 0)
 			(hide yes)
@@
 			)
 		)
-		(property "Value" "47k"
+		(property "Value" "47k 1%"
 			(at 120.65 92.71 0)
 			(show_name no)

Commit message: Align I2C resistors for 100kHZ ops.
Parts:
- R19, R20: value 4.7k -> 2.2k; LCSC (none) -> C4190; now fitted; now in the parts list
Changed lines of the file:
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@@
 		(body_style 1)
 		(exclude_from_sim no)
-		(in_bom no)
-		(on_board yes)
-		(in_pos_files yes)
-		(dnp yes)
+		(in_bom yes)
+		(on_board yes)
+		(in_pos_files yes)
+		(dnp no)
 		(property "Reference" "R19"
 			(at 217.17 92.71 0)
@@
 			)
 		)
-		(property "Value" "4.7k"
+		(property "Value" "2.2k"
 			(at 217.17 95.25 0)
 			(show_name no)
@@
 		)
 		(property "Description" "Resistor"
+			(at 215.9 93.98 0)
+			(hide yes)
+			(show_name no)
+			(do_not_autoplace no)
+			(effects
+				(font
+					(size 1.27 1.27)
+				)
+			)
+		)
+		(property "LCSC" "C4190"
 			(at 215.9 93.98 0)
 			(hide yes)
@@
 		(body_style 1)
 		(exclude_from_sim no)
-		(in_bom no)
-		(on_board yes)
-		(in_pos_files yes)
-		(dnp yes)
+		(in_bom yes)
+		(on_board yes)
+		(in_pos_files yes)
+		(dnp no)
 		(property "Reference" "R20"
 			(at 240.03 92.71 0)
@@
 			)
 		)
-		(property "Value" "4.7k"
+		(property "Value" "2.2k"
 			(at 240.03 95.25 0)
 			(show_name no)
@@
 			(at 238.76 93.98 0)
 			(hide yes)
+			(show_name no)
+			(do_not_autoplace no)
+			(effects
+				(font
+					(size 1.27 1.27)
+				)
+			)
+		)
+		(property "LCSC" "C4190"
+			(at 238.76 93.98 0)
+			(hide yes)

Commit message: Other MH's.
Connections:
- net ESP_3V3 renamed +ESP_3V3
- net RAIL_5V renamed +5V
- net VBAT renamed +VBAT
- net VSYS renamed +VSYS
Changed lines of the file:
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@@
 	)
 	(symbol
-		(lib_id "carrier:ESP_3V3")
+		(lib_id "carrier:+ESP_3V3")
 		(at 227.33 86.36 0)
 		(unit 1)
@@
 			)
 		)
-		(property "Value" "ESP_3V3"
+		(property "Value" "+ESP_3V3"
 			(at 227.33 82.55 0)
 			(show_name no)
@@
 			)
 		)
-		(property "Description" "Power symbol creates a global label with name \"ESP_3V3\""
+		(property "Description" "Power symbol creates a global label with name \"+ESP_3V3\""
 			(at 227.33 86.36 0)
 			(hide yes)
@@
 	)
 	(symbol
-		(lib_id "carrier:RAIL_5V")
+		(lib_id "carrier:+5V")
 		(at 152.4 86.36 0)
 		(unit 1)
@@
 			)
 		)
-		(property "Value" "RAIL_5V"
+		(property "Value" "+5V"
 			(at 152.4 82.55 0)
 			(show_name no)
@@
 			)
 		)
-		(property "Description" "Power symbol creates a global label with name \"RAIL_5V\""
+		(property "Description" "Power symbol creates a global label with name \"+5V\""
 			(at 152.4 86.36 0)
 			(hide yes)
@@
 	)
 	(symbol
-		(lib_id "carrier:VBAT")
+		(lib_id "carrier:+VBAT")
 		(at 165.1 81.28 0)
 		(unit 1)
@@
 			)
 		)
-		(property "Value" "VBAT"
+		(property "Value" "+VBAT"
 			(at 165.1 77.47 0)
 			(show_name no)
@@
 			)
 		)
-		(property "Description" "Power symbol creates a global label with name \"VBAT\""
+		(property "Description" "Power symbol creates a global label with name \"+VBAT\""
 			(at 165.1 81.28 0)
 			(hide yes)
@@
 	)
 	(symbol
-		(lib_id "carrier:VSYS")
+		(lib_id "carrier:+VSYS")
 		(at 102.87 86.36 0)
 		(unit 1)
@@
 			)
 		)
-		(property "Value" "VSYS"
+		(property "Value" "+VSYS"
 			(at 102.87 82.55 0)
 			(show_name no)
@@
 			)
 		)
-		(property "Description" "Power symbol creates a global label with name \"VSYS\""
+		(property "Description" "Power symbol creates a global label with name \"+VSYS\""
 			(at 102.87 86.36 0)
 			(hide yes)

Commit message: Add USB current detection.
Changed lines of the file:
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@@
 	)
 	(global_label "I2C_SCL"
-		(shape bidirectional)
+		(shape input)
 		(at 241.3 104.14 0)
 		(effects

Commit message: Switch to faster FUSB303B USB controller.
Parts:
- R19, R20: value 2.2k -> 1.8k; LCSC C4190 -> C4177
Changed lines of the file:
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@@
 			)
 		)
-		(property "Value" "2.2k"
+		(property "Value" "1.8k"
 			(at 217.17 95.25 0)
 			(show_name no)
@@
 			)
 		)
-		(property "LCSC" "C4190"
+		(property "LCSC" "C4177"
 			(at 215.9 93.98 0)
 			(hide yes)
@@
 			)
 		)
-		(property "Value" "2.2k"
+		(property "Value" "1.8k"
 			(at 240.03 95.25 0)
 			(show_name no)
@@
 			)
 		)
-		(property "LCSC" "C4190"
+		(property "LCSC" "C4177"
 			(at 238.76 93.98 0)
 			(hide yes)

Commit message: Consolidate bom.
Parts:
- C27: value 100n 50V -> 100n 16V; footprint Capacitor_SMD:C_0603_1608Metric -> carrier:C_0402_1005Metric_NoSilk; LCSC C14663 -> C1525; MPN (none) -> CL05B104KO5NNNC
Changed lines of the file:
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@@
 			)
 		)
-		(property "Value" "100n 50V"
+		(property "Value" "100n 16V"
 			(at 175.26 90.17 0)
 			(show_name no)
@@
 			)
 		)
-		(property "Footprint" "Capacitor_SMD:C_0603_1608Metric"
+		(property "Footprint" "carrier:C_0402_1005Metric_NoSilk"
 			(at 172.72 88.9 0)
 			(hide yes)
@@
 			)
 		)
-		(property "LCSC" "C14663"
+		(property "LCSC" "C1525"
 			(at 172.72 88.9 0)
 			(hide yes)
+			(show_name no)
+			(do_not_autoplace no)
+			(effects
+				(font
+					(size 1.27 1.27)
+				)
+			)
+		)
+		(property "MPN" "CL05B104KO5NNNC"
+			(at 172.72 88.9 0)
+			(hide yes)

Commit message: Polishing.
Parts:
- added R90, R91: 5.1k, Resistor_SMD:R_0805_2012Metric_Pad1.20x1.40mm_HandSolder, symbol Device:R
- R19, R20: value 1.8k -> 1.43k; LCSC C4177 -> C22840; MPN (none) -> 0603WAF1431T5E; Manufacturer (none) -> UNI-ROYAL; Tolerance (none) -> 1%
Connections:
- net +ESP_3V3: now also R90.1, R91.1
- net I2C_SCL: now also R91.2
- net I2C_SDA: now also R90.2
Changed lines of the file:
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@@
 			)
 		)
-		(property "Value" "1.8k"
+		(property "Value" "1.43k"
 			(at 217.17 95.25 0)
 			(show_name no)
@@
 			)
 		)
-		(property "Datasheet" ""
+		(property "Datasheet" "https://datasheet.lcsc.com/datasheet/pdf/0a975aaa49b7c97f38a963127be4a823.pdf?productCode=C22840"
 			(at 215.9 93.98 0)
 			(hide yes)
@@
 			)
 		)
-		(property "LCSC" "C4177"
+		(property "LCSC" "C22840"
 			(at 215.9 93.98 0)
 			(hide yes)
@@
 			)
 		)
+		(property "MPN" "0603WAF1431T5E" (at 215.9 93.98 0) (hide yes) (effects (font (size 1.27 1.27))))
+		(property "Manufacturer" "UNI-ROYAL" (at 215.9 93.98 0) (hide yes) (effects (font (size 1.27 1.27))))
+		(property "Tolerance" "1%" (at 215.9 93.98 0) (hide yes) (effects (font (size 1.27 1.27))))
 	)
 	(symbol
@@
 			)
 		)
-		(property "Value" "1.8k"
+		(property "Value" "1.43k"
 			(at 240.03 95.25 0)
 			(show_name no)
@@
 			)
 		)
-		(property "Datasheet" ""
+		(property "Datasheet" "https://datasheet.lcsc.com/datasheet/pdf/0a975aaa49b7c97f38a963127be4a823.pdf?productCode=C22840"
 			(at 238.76 93.98 0)
 			(hide yes)
@@
 			)
 		)
-		(property "LCSC" "C4177"
+		(property "LCSC" "C22840"
 			(at 238.76 93.98 0)
 			(hide yes)
@@
 			)
 		)
+		(property "MPN" "0603WAF1431T5E" (at 238.76 93.98 0) (hide yes) (effects (font (size 1.27 1.27))))
+		(property "Manufacturer" "UNI-ROYAL" (at 238.76 93.98 0) (hide yes) (effects (font (size 1.27 1.27))))
+		(property "Tolerance" "1%" (at 238.76 93.98 0) (hide yes) (effects (font (size 1.27 1.27))))
 	)
 	(symbol
@@
 		)
 	)
+	(symbol
+		(lib_id "Device:R")
+		(at 215.9000 116.8400 0)
+		(unit 1)
+		(body_style 1)
+		(exclude_from_sim no)
+		(in_bom no)
+		(on_board yes)
+		(in_pos_files no)
+		(dnp yes)
+		(property "Reference" "R90"
+			(at 217.1700 115.5700 0)
+			(show_name no)
+			(do_not_autoplace no)
+			(effects
+				(font
+					(size 1.27 1.27)
+				)
+				(justify left)
+			)
+		)
+		(property "Value" "5.1k"
+			(at 217.1700 118.1100 0)
+			(show_name no)
+			(do_not_autoplace no)
+			(effects
+				(font
+					(size 1.27 1.27)
+				)
+				(justify left)
+			)
+		)
+		(property "Footprint" "Resistor_SMD:R_0805_2012Metric_Pad1.20x1.40mm_HandSolder"
+			(at 215.9000 116.8400 0)
+			(hide yes)
+			(show_name no)
+			(do_not_autoplace no)
+			(effects
+				(font
+					(size 1.27 1.27)
+				)
+			)
+		)
+		(property "Datasheet" ""
+			(at 215.9000 116.8400 0)
+			(hide yes)
+			(show_name no)
+			(do_not_autoplace no)
+			(effects
+				(font
+					(size 1.27 1.27)
+				)
+			)
+		)
+		(property "Description" "Optional parallel I2C_SDA pull-up, fit only after measuring the bus"
+			(at 215.9000 116.8400 0)
+			(hide yes)
+			(show_name no)
+			(do_not_autoplace no)
+			(effects
+				(font
+					(size 1.27 1.27)
+				)
+			)
+		)
+		(pin "1"
+		)
+		(pin "2"
+		)
+		(instances
+			(project "carrier"
+				(path "/1d76d2ec-7795-4c71-8167-b1182c3ebc1d/f622a697-5a21-4794-a4ab-94e63edd90cd"
+					(reference "R90")
+					(unit 1)
+				)
+			)
+		)
+	)
+	(global_label "+ESP_3V3" (shape bidirectional) (at 215.9000 113.0300 0) (effects (font (size 1.27 1.27)) (justify left)))
+	(global_label "I2C_SDA" (shape bidirectional) (at 215.9000 120.6500 0) (effects (font (size 1.27 1.27)) (justify left)))
+	(symbol
+		(lib_id "Device:R")
+		(at 238.7600 116.8400 0)
+		(unit 1)
+		(body_style 1)
+		(exclude_from_sim no)
+		(in_bom no)
+		(on_board yes)
+		(in_pos_files no)
+		(dnp yes)
+		(property "Reference" "R91"
+			(at 240.0300 115.5700 0)
+			(show_name no)
+			(do_not_autoplace no)
+			(effects
+				(font
+					(size 1.27 1.27)
+				)
+				(justify left)
+			)
+		)
+		(property "Value" "5.1k"
+			(at 240.0300 118.1100 0)
+			(show_name no)
+			(do_not_autoplace no)
+			(effects
+				(font
+					(size 1.27 1.27)
+				)
+				(justify left)
+			)
+		)
+		(property "Footprint" "Resistor_SMD:R_0805_2012Metric_Pad1.20x1.40mm_HandSolder"
+			(at 238.7600 116.8400 0)
+			(hide yes)
+			(show_name no)
+			(do_not_autoplace no)
+			(effects
+				(font
+					(size 1.27 1.27)
+				)
+			)
+		)
+		(property "Datasheet" ""
+			(at 238.7600 116.8400 0)
+			(hide yes)
+			(show_name no)
+			(do_not_autoplace no)
+			(effects
+				(font
+					(size 1.27 1.27)
+				)
+			)
+		)
+		(property "Description" "Optional parallel I2C_SCL pull-up, fit only after measuring the bus"
+			(at 238.7600 116.8400 0)
+			(hide yes)
+			(show_name no)
+			(do_not_autoplace no)
+			(effects
+				(font
+					(size 1.27 1.27)
+				)
+			)
+		)
+		(pin "1"
+		)
+		(pin "2"
+		)
+		(instances
+			(project "carrier"
+				(path "/1d76d2ec-7795-4c71-8167-b1182c3ebc1d/f622a697-5a21-4794-a4ab-94e63edd90cd"
+					(reference "R91")
+					(unit 1)
+				)
+			)
+		)
+	)
+	(global_label "+ESP_3V3" (shape bidirectional) (at 238.7600 113.0300 0) (effects (font (size 1.27 1.27)) (justify left)))
+	(global_label "I2C_SCL" (shape bidirectional) (at 238.7600 120.6500 0) (effects (font (size 1.27 1.27)) (justify left)))
 )

Commit message: Consolidate BOM, add GNSS listen to ESP.
Parts:
- C27: footprint carrier:C_0402_1005Metric_NoSilk -> Mark:C_0402_1005Metric_NoSilk
- D3: renamed from D5; footprint carrier:LED_D3.0mm -> Mark:LED_D3.0mm
- R19, R20: value 1.43k -> 1.5k; LCSC C22840 -> C22843; MPN 0603WAF1431T5E -> 0603WAF1501T5E
- U8: footprint carrier:TDFN-8_L2.0-W2.0-P0.50-EP0.8x1.38_T822 -> Mark:TDFN-8_L2.0-W2.0-P0.50-EP0.8x1.38_T822; symbol carrier:MAX17048G+T10 -> Mark:MAX17048G+T10
- renumbered D4 to D2
