File: hardware/carrier-ti-charger/usb_input.kicad_sch (KiCad schematic)
At the start: 11 parts, among them J1 MC-107DMS, U15 FUSB303BTMX

Commit message: Polishing.
Parts:
- renumbered J1 to J14
Changed lines of the file:
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@@
 		(in_pos_files yes)
 		(dnp no)
-		(property "Reference" "J1"
+		(property "Reference" "J14"
 			(at 35.56 67.31 0)
 			(show_name no)
@@
 			(project "carrier"
 				(path "/1d76d2ec-7795-4c71-8167-b1182c3ebc1d/8d582056-b074-472b-a300-fd21b59a9139"
-					(reference "J1")
+					(reference "J14")
 					(unit 1)
 				)

Commit message: Consolidate BOM, add GNSS listen to ESP.
Parts:
- C57: footprint carrier:C_0402_1005Metric_NoSilk -> Mark:C_0402_1005Metric_NoSilk
- J14: footprint carrier:USB_C_Receptacle_Hanbo_MC-107DMS -> Mark:USB_C_Receptacle_Hanbo_MC-107DMS
- R79, R80, R81: footprint carrier:R_0402_1005Metric_NoSilk -> Mark:R_0402_1005Metric_NoSilk
- U15: footprint carrier:X2QFN-12_L1.6-W1.6-P0.40-TL -> Mark:X2QFN-12_L1.6-W1.6-P0.40-TL; symbol carrier:FUSB303BTMX -> Mark:FUSB303BTMX
- renumbered D3 to D1, D8 to D4, D9 to D5
Changed lines of the file:
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@@
 			)
 		)
-		(property "Footprint" "carrier:R_0402_1005Metric_NoSilk"
+		(property "Footprint" "Mark:R_0402_1005Metric_NoSilk"
 			(at 180.34 116.84 0)
 			(hide yes)
@@
 			)
 		)
-		(property "Footprint" "carrier:R_0402_1005Metric_NoSilk"
+		(property "Footprint" "Mark:R_0402_1005Metric_NoSilk"
 			(at 160.02 116.84 0)
 			(hide yes)
@@
 	)
 	(symbol
-		(lib_id "carrier:+VUSB")
+		(lib_id "Mark:+VUSB")
 		(at 170.18 120.65 180)
 		(unit 1)
@@
 	)
 	(symbol
-		(lib_id "carrier:FUSB303BTMX")
+		(lib_id "Mark:FUSB303BTMX")
 		(at 177.8 85.09 0)
 		(unit 1)
@@
 			)
 		)
-		(property "Footprint" "carrier:X2QFN-12_L1.6-W1.6-P0.40-TL"
+		(property "Footprint" "Mark:X2QFN-12_L1.6-W1.6-P0.40-TL"
 			(at 177.8 85.09 0)
 			(hide yes)
@@
 			)
 		)
-		(property "Footprint" "carrier:C_0402_1005Metric_NoSilk"
+		(property "Footprint" "Mark:C_0402_1005Metric_NoSilk"
 			(at 208.28 77.47 0)
 			(hide yes)
@@
 		(in_pos_files yes)
 		(dnp no)
-		(property "Reference" "D3"
+		(property "Reference" "D1"
 			(at 88.9 59.69 90)
 			(show_name no)
@@
 			(project "carrier"
 				(path "/1d76d2ec-7795-4c71-8167-b1182c3ebc1d/8d582056-b074-472b-a300-fd21b59a9139"
-					(reference "D3")
+					(reference "D1")
 					(unit 1)
 				)
@@
 	)
 	(symbol
-		(lib_id "carrier:+VUSB")
+		(lib_id "Mark:+VUSB")
 		(at 114.3 53.34 0)
 		(unit 1)
@@
 			)
 		)
-		(property "Footprint" "carrier:R_0402_1005Metric_NoSilk"
+		(property "Footprint" "Mark:R_0402_1005Metric_NoSilk"
 			(at 170.18 116.84 0)
 			(hide yes)
@@
 	)
 	(symbol
-		(lib_id "carrier:+ESP_3V3")
+		(lib_id "Mark:+ESP_3V3")
 		(at 200.66 71.12 0)
 		(unit 1)
@@
 			)
 		)
-		(property "Footprint" "carrier:USB_C_Receptacle_Hanbo_MC-107DMS"
+		(property "Footprint" "Mark:USB_C_Receptacle_Hanbo_MC-107DMS"
 			(at 45.72 88.9 0)
 			(hide yes)
@@
 		(in_pos_files yes)
 		(dnp no)
-		(property "Reference" "D9"
+		(property "Reference" "D5"
 			(at 91.44 102.87 90)
 			(show_name no)
@@
 			(project "carrier"
 				(path "/1d76d2ec-7795-4c71-8167-b1182c3ebc1d/8d582056-b074-472b-a300-fd21b59a9139"
-					(reference "D9")
+					(reference "D5")
 					(unit 1)
 				)
@@
 		(in_pos_files yes)
 		(dnp no)
-		(property "Reference" "D8"
+		(property "Reference" "D4"
 			(at 71.12 102.87 90)
 			(show_name no)
@@
 			(project "carrier"
 				(path "/1d76d2ec-7795-4c71-8167-b1182c3ebc1d/8d582056-b074-472b-a300-fd21b59a9139"
-					(reference "D8")
-					(unit 1)
-				)
+					(reference "D4")
+					(unit 1)
+				)
