File: hardware/insulator/insulator.kicad_pcb (KiCad board)
At the start: 2 copper layers, 105 x 95 mm, 8 parts

Commit message: Polishing.
Other:
- board text added: "J11"
- board text added: "J12"
- board text added: "J13"
- board text removed: "J2"
- board text removed: "J3"
- board text removed: "J4"
Changed lines of the file:
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@@
 		(layer "Edge.Cuts")
 	)
-	(gr_text "J3"
+	(gr_text "J11"
 		(at 41.418 73.049 0)
 		(layer "F.SilkS")
@@
 		)
 	)
-	(gr_text "J4"
+	(gr_text "J13"
 		(at 41.656 88.791 0)
 		(layer "F.SilkS")
@@
 		)
 	)
-	(gr_text "J2"
+	(gr_text "J12"
 		(at 48.742 73.033 0)
 		(layer "F.SilkS")

Commit message: Order revision A.
Parts:
- removed MH6, MH7, MH8: antenna clearance 11 mm, 
- added MH6ANTGNSS: antenna clearance 11 mm, , F.Cu at (31.5, 7.80)
- added MH7ADS1090: antenna clearance 11 mm, , F.Cu at (50.5, 7.80)
- added MH8ADS980: antenna clearance 11 mm, , F.Cu at (74.1, 7.80)
- added REF**: OSHW-Logo_7.5x8mm_SilkScreen, Symbol:OSHW-Logo_7.5x8mm_SilkScreen, B.Cu at (88.4, 35.7)
- MH1, MH2, MH3, MH4: value MountingHole_2.7mm_M2.5 -> MountingHole_2.7mm_M2.5_Pad_Via; footprint MountingHole:MountingHole_2.7mm_M2.5 -> MountingHole:MountingHole_2.7mm_M2.5_Pad_Via
- moved MH2 0.78 mm to (101.0, 4.02)
- moved MH4 0.75 mm to (101.0, 91.0)
- moved MH1 0.63 mm to (3.99, 4.02)
- moved MH3 0.63 mm to (3.98, 91.0)
- moved H1 0.13 mm to (45.0, 80.9)
Other:
- board text added: "CABLES"
- board text added: "Rev A 2026-10-19"
- board text removed: "CARRIER INSULATOR Rev A 2026-10-03"
- board text removed: "J11"
- board text removed: "J12"
- board text removed: "J13"
